File: KiCad/prot2/prot2.kicad_pcb (KiCad board)
At the start: 2 copper layers, 1 part, among them Q1 Q_Photo_NPN

Commit message: ネジ穴配置
Parts:
- added C1: C, Capacitor_SMD:C_0603_1608Metric_Pad1.08x0.95mm_HandSolder, F.Cu at (32.0, 45.1)
- added C10: C, Capacitor_SMD:C_0603_1608Metric_Pad1.08x0.95mm_HandSolder, F.Cu at (32.0, 67.7)
- added C11: C_Polarized_Small_US, Package_SO:SOIC-14_3.9x8.7mm_P1.27mm, F.Cu at (71.9, 79.2)
- added C12: C_Polarized_Small_US, Capacitor_THT:C_Radial_D8.0mm_H11.5mm_P3.50mm, F.Cu at (96.0, 78.7)
- added C13: C_Polarized_Small_US, Capacitor_THT:C_Radial_D8.0mm_H11.5mm_P3.50mm, F.Cu at (96.0, 88.3)
- added C2: C, Capacitor_SMD:C_0603_1608Metric_Pad1.08x0.95mm_HandSolder, F.Cu at (32.0, 47.6)
- added C3: C, Capacitor_SMD:C_0603_1608Metric_Pad1.08x0.95mm_HandSolder, F.Cu at (32.0, 50.1)
- added C4: C, Capacitor_SMD:C_0603_1608Metric_Pad1.08x0.95mm_HandSolder, F.Cu at (32.0, 52.6)
- added C5: C, Capacitor_SMD:C_0603_1608Metric_Pad1.08x0.95mm_HandSolder, F.Cu at (32.0, 55.1)
- added C6: C, Capacitor_SMD:C_0603_1608Metric_Pad1.08x0.95mm_HandSolder, F.Cu at (32.0, 57.6)
- added C7: C, Capacitor_SMD:C_0603_1608Metric_Pad1.08x0.95mm_HandSolder, F.Cu at (32.0, 60.1)
- added C8: C, Capacitor_SMD:C_0603_1608Metric_Pad1.08x0.95mm_HandSolder, F.Cu at (32.0, 62.6)
- added C9: C, Capacitor_SMD:C_0603_1608Metric_Pad1.08x0.95mm_HandSolder, F.Cu at (32.0, 65.1)
- added D1: LED, LED_SMD:LED_0603_1608Metric_Pad1.05x0.95mm_HandSolder, F.Cu at (71.2, 45.1)
- added D10: LED, LED_SMD:LED_0603_1608Metric_Pad1.05x0.95mm_HandSolder, F.Cu at (75.6, 45.1)
- added D11: LED, LED_SMD:LED_0603_1608Metric_Pad1.05x0.95mm_HandSolder, F.Cu at (75.6, 47.7)
- added D12: LED, LED_SMD:LED_0603_1608Metric_Pad1.05x0.95mm_HandSolder, F.Cu at (75.6, 50.3)
- added D13: LED, LED_SMD:LED_0603_1608Metric_Pad1.05x0.95mm_HandSolder, F.Cu at (75.6, 52.9)
- added D14: LED, LED_SMD:LED_0603_1608Metric_Pad1.05x0.95mm_HandSolder, F.Cu at (75.6, 55.5)
- added D15: LED, LED_SMD:LED_0603_1608Metric_Pad1.05x0.95mm_HandSolder, F.Cu at (75.6, 58.1)
- added D16: LED, LED_SMD:LED_0603_1608Metric_Pad1.05x0.95mm_HandSolder, F.Cu at (75.6, 60.6)
- added D17: LED, LED_SMD:LED_0603_1608Metric_Pad1.05x0.95mm_HandSolder, F.Cu at (75.6, 63.2)
- added D18: LED, LED_SMD:LED_0603_1608Metric_Pad1.05x0.95mm_HandSolder, F.Cu at (75.6, 65.8)
- added D19: LED, LED_SMD:LED_0603_1608Metric_Pad1.05x0.95mm_HandSolder, F.Cu at (80.0, 45.1)
- added D2: LED, LED_SMD:LED_0603_1608Metric_Pad1.05x0.95mm_HandSolder, F.Cu at (71.2, 47.7)
- added D20: LED, LED_SMD:LED_0603_1608Metric_Pad1.05x0.95mm_HandSolder, F.Cu at (80.0, 47.7)
- added D21: LED, LED_SMD:LED_0603_1608Metric_Pad1.05x0.95mm_HandSolder, F.Cu at (80.0, 50.3)
- added D22: LED, LED_SMD:LED_0603_1608Metric_Pad1.05x0.95mm_HandSolder, F.Cu at (80.0, 52.9)
- added D23: LED, LED_SMD:LED_0603_1608Metric_Pad1.05x0.95mm_HandSolder, F.Cu at (80.0, 55.5)
- added D24: LED, LED_SMD:LED_0603_1608Metric_Pad1.05x0.95mm_HandSolder, F.Cu at (80.0, 58.1)
- added D25: LED, LED_SMD:LED_0603_1608Metric_Pad1.05x0.95mm_HandSolder, F.Cu at (80.0, 60.6)
- added D26: LED, LED_SMD:LED_0603_1608Metric_Pad1.05x0.95mm_HandSolder, F.Cu at (80.0, 63.2)
- added D27: LED, LED_SMD:LED_0603_1608Metric_Pad1.05x0.95mm_HandSolder, F.Cu at (80.0, 65.8)
- added D28: LED, LED_SMD:LED_0603_1608Metric_Pad1.05x0.95mm_HandSolder, F.Cu at (84.4, 45.1)
- added D29: LED, LED_SMD:LED_0603_1608Metric_Pad1.05x0.95mm_HandSolder, F.Cu at (84.4, 47.7)
- added D3: LED, LED_SMD:LED_0603_1608Metric_Pad1.05x0.95mm_HandSolder, F.Cu at (71.2, 50.3)
- added D30: LED, LED_SMD:LED_0603_1608Metric_Pad1.05x0.95mm_HandSolder, F.Cu at (84.4, 50.3)
- added D31: LED, LED_SMD:LED_0603_1608Metric_Pad1.05x0.95mm_HandSolder, F.Cu at (84.4, 52.9)
- added D32: LED, LED_SMD:LED_0603_1608Metric_Pad1.05x0.95mm_HandSolder, F.Cu at (84.4, 55.5)
- added D33: D_Schottky, Diode_SMD:D_SOD-323_HandSoldering, F.Cu at (98.6, 59.0)
- added D4: LED, LED_SMD:LED_0603_1608Metric_Pad1.05x0.95mm_HandSolder, F.Cu at (71.2, 52.9)
- added D5: LED, LED_SMD:LED_0603_1608Metric_Pad1.05x0.95mm_HandSolder, F.Cu at (71.2, 55.5)
- added D6: LED, LED_SMD:LED_0603_1608Metric_Pad1.05x0.95mm_HandSolder, F.Cu at (71.2, 58.1)
- added D7: LED, LED_SMD:LED_0603_1608Metric_Pad1.05x0.95mm_HandSolder, F.Cu at (71.2, 60.6)
- added D8: LED, LED_SMD:LED_0603_1608Metric_Pad1.05x0.95mm_HandSolder, F.Cu at (71.2, 63.2)
- added D9: LED, LED_SMD:LED_0603_1608Metric_Pad1.05x0.95mm_HandSolder, F.Cu at (71.2, 65.8)
- added H1: MountingHole, MountingHole:MountingHole_3.2mm_M3, F.Cu at (551.6, 551.6)
- added H2: MountingHole, MountingHole:MountingHole_3.2mm_M3, F.Cu at (551.6, 448.4)
- added H3: MountingHole, MountingHole:MountingHole_3.2mm_M3, F.Cu at (448.4, 551.6)
- added H4: MountingHole, MountingHole:MountingHole_3.2mm_M3, F.Cu at (448.4, 448.4)
- added J1: Conn_01x02_Socket, Connector_JST:JST_XH_S2B-XH-A_1x02_P2.50mm_Horizontal, F.Cu at (90.1, 60.9)
- added J2: LED_SW, Connector_PinHeader_2.54mm:PinHeader_1x03_P2.54mm_Vertical, F.Cu at (62.1, 101.5)
- added J3: Conn_01x04_Socket, Connector_JST:JST_PH_S4B-PH-K_1x04_P2.00mm_Horizontal, F.Cu at (50.8, 101.5)
- added LS1: Speaker_Crystal, Buzzer_Beeper:Buzzer_TDK_PS1240P02BT_D12.2mm_H6.5mm, F.Cu at (91.2, 50.7)
- added Q10: Q_Photo_NPN, NJL7502R:NJL7502R, F.Cu at (31.0, 103.1)
- added Q11: Q_Photo_NPN, NJL7502R:NJL7502R, F.Cu at (33.2, 103.1)
- added Q12: Q_Photo_NPN, NJL7502R:NJL7502R, F.Cu at (35.5, 103.1)
- added Q13: Q_Photo_NPN, NJL7502R:NJL7502R, F.Cu at (37.7, 103.1)
- added Q14: Q_Photo_NPN, NJL7502R:NJL7502R, F.Cu at (40.0, 103.1)
- added Q15: Q_Photo_NPN, NJL7502R:NJL7502R, F.Cu at (42.2, 103.1)
- added Q16: Q_Photo_NPN, NJL7502R:NJL7502R, F.Cu at (44.5, 103.1)
- added Q17: Q_Photo_NPN, NJL7502R:NJL7502R, F.Cu at (46.7, 103.1)
- added Q18: Q_Photo_NPN, NJL7502R:NJL7502R, F.Cu at (31.0, 105.7)
- added Q19: Q_Photo_NPN, NJL7502R:NJL7502R, F.Cu at (33.2, 105.7)
- added Q2: Q_Photo_NPN, NJL7502R:NJL7502R, F.Cu at (31.0, 100.5)
- added Q20: Q_Photo_NPN, NJL7502R:NJL7502R, F.Cu at (35.5, 105.7)
- added Q21: Q_Photo_NPN, NJL7502R:NJL7502R, F.Cu at (37.7, 105.7)
- added Q22: Q_Photo_NPN, NJL7502R:NJL7502R, F.Cu at (40.0, 105.7)
- added Q23: Q_Photo_NPN, NJL7502R:NJL7502R, F.Cu at (42.2, 105.7)
- added Q24: Q_Photo_NPN, NJL7502R:NJL7502R, F.Cu at (44.5, 105.7)
- added Q25: Q_Photo_NPN, NJL7502R:NJL7502R, F.Cu at (46.7, 105.7)
- added Q26: Q_Photo_NPN, NJL7502R:NJL7502R, F.Cu at (31.0, 108.3)
- added Q27: Q_Photo_NPN, NJL7502R:NJL7502R, F.Cu at (33.2, 108.3)
- added Q28: Q_Photo_NPN, NJL7502R:NJL7502R, F.Cu at (35.5, 108.3)
- added Q29: Q_Photo_NPN, NJL7502R:NJL7502R, F.Cu at (37.7, 108.3)
- added Q3: Q_Photo_NPN, NJL7502R:NJL7502R, F.Cu at (33.2, 100.5)
- added Q30: Q_Photo_NPN, NJL7502R:NJL7502R, F.Cu at (40.0, 108.3)
- added Q31: Q_Photo_NPN, NJL7502R:NJL7502R, F.Cu at (42.2, 108.3)
- added Q32: Q_Photo_NPN, NJL7502R:NJL7502R, F.Cu at (44.5, 108.3)
- added Q4: Q_Photo_NPN, NJL7502R:NJL7502R, F.Cu at (35.5, 100.5)
- added Q5: Q_Photo_NPN, NJL7502R:NJL7502R, F.Cu at (37.7, 100.5)
- added Q6: Q_Photo_NPN, NJL7502R:NJL7502R, F.Cu at (40.0, 100.5)
- added Q7: Q_Photo_NPN, NJL7502R:NJL7502R, F.Cu at (42.2, 100.5)
- added Q8: Q_Photo_NPN, NJL7502R:NJL7502R, F.Cu at (44.5, 100.5)
- added Q9: Q_Photo_NPN, NJL7502R:NJL7502R, F.Cu at (46.7, 100.5)
- added RP2040_Zero1: ~, RP2040zero:RP2040_zero, F.Cu at (39.3, 77.0)
- added RP2040_Zero2: ~, RP2040zero:RP2040_zero, F.Cu at (58.2, 77.0)
- added RV1: R_Potentiometer_Trim, hankotei:hankotei_node, F.Cu at (97.5, 106.7)
- added Rc1: R, Resistor_SMD:R_0603_1608Metric_Pad0.98x0.95mm_HandSolder, F.Cu at (32.0, 70.2)
- added Rc10: R, Resistor_SMD:R_0603_1608Metric_Pad0.98x0.95mm_HandSolder, F.Cu at (36.4, 62.6)
- added Rc11: R, Resistor_SMD:R_0603_1608Metric_Pad0.98x0.95mm_HandSolder, F.Cu at (36.4, 65.1)
- added Rc12: R, Resistor_SMD:R_0603_1608Metric_Pad0.98x0.95mm_HandSolder, F.Cu at (36.4, 67.7)
- added Rc13: R, Resistor_SMD:R_0603_1608Metric_Pad0.98x0.95mm_HandSolder, F.Cu at (36.4, 70.2)
- added Rc14: R, Resistor_SMD:R_0603_1608Metric_Pad0.98x0.95mm_HandSolder, F.Cu at (36.4, 72.7)
- added Rc15: R, Resistor_SMD:R_0603_1608Metric_Pad0.98x0.95mm_HandSolder, F.Cu at (40.7, 45.1)
- added Rc16: R, Resistor_SMD:R_0603_1608Metric_Pad0.98x0.95mm_HandSolder, F.Cu at (40.7, 47.6)
- added Rc17: R, Resistor_SMD:R_0603_1608Metric_Pad0.98x0.95mm_HandSolder, F.Cu at (40.7, 50.1)
- added Rc18: R, Resistor_SMD:R_0603_1608Metric_Pad0.98x0.95mm_HandSolder, F.Cu at (40.7, 52.6)
- added Rc19: R, Resistor_SMD:R_0603_1608Metric_Pad0.98x0.95mm_HandSolder, F.Cu at (40.7, 55.1)
- added Rc2: R, Resistor_SMD:R_0603_1608Metric_Pad0.98x0.95mm_HandSolder, F.Cu at (32.0, 72.7)
- added Rc20: R, Resistor_SMD:R_0603_1608Metric_Pad0.98x0.95mm_HandSolder, F.Cu at (40.7, 57.6)
- added Rc21: R, Resistor_SMD:R_0603_1608Metric_Pad0.98x0.95mm_HandSolder, F.Cu at (40.7, 60.1)
- added Rc22: R, Resistor_SMD:R_0603_1608Metric_Pad0.98x0.95mm_HandSolder, F.Cu at (40.7, 62.6)
- added Rc23: R, Resistor_SMD:R_0603_1608Metric_Pad0.98x0.95mm_HandSolder, F.Cu at (40.7, 65.1)
- added Rc24: R, Resistor_SMD:R_0603_1608Metric_Pad0.98x0.95mm_HandSolder, F.Cu at (40.7, 67.7)
- added Rc25: R, Resistor_SMD:R_0603_1608Metric_Pad0.98x0.95mm_HandSolder, F.Cu at (40.7, 70.2)
- added Rc26: R, Resistor_SMD:R_0603_1608Metric_Pad0.98x0.95mm_HandSolder, F.Cu at (40.7, 72.7)
- added Rc27: R, Resistor_SMD:R_0603_1608Metric_Pad0.98x0.95mm_HandSolder, F.Cu at (45.1, 45.1)
- added Rc28: R, Resistor_SMD:R_0603_1608Metric_Pad0.98x0.95mm_HandSolder, F.Cu at (45.1, 47.6)
- added Rc29: R, Resistor_SMD:R_0603_1608Metric_Pad0.98x0.95mm_HandSolder, F.Cu at (45.1, 50.1)
- added Rc3: R, Resistor_SMD:R_0603_1608Metric_Pad0.98x0.95mm_HandSolder, F.Cu at (36.4, 45.1)
- added Rc30: R, Resistor_SMD:R_0603_1608Metric_Pad0.98x0.95mm_HandSolder, F.Cu at (45.1, 52.6)
- added Rc31: R, Resistor_SMD:R_0603_1608Metric_Pad0.98x0.95mm_HandSolder, F.Cu at (45.1, 55.1)
- added Rc32: R, Resistor_SMD:R_0603_1608Metric_Pad0.98x0.95mm_HandSolder, F.Cu at (45.1, 57.6)
- added Rc4: R, Resistor_SMD:R_0603_1608Metric_Pad0.98x0.95mm_HandSolder, F.Cu at (36.4, 47.6)
- added Rc5: R, Resistor_SMD:R_0603_1608Metric_Pad0.98x0.95mm_HandSolder, F.Cu at (36.4, 50.1)
- added Rc6: R, Resistor_SMD:R_0603_1608Metric_Pad0.98x0.95mm_HandSolder, F.Cu at (36.4, 52.6)
- added Rc7: R, Resistor_SMD:R_0603_1608Metric_Pad0.98x0.95mm_HandSolder, F.Cu at (36.4, 55.1)
- added Rc8: R, Resistor_SMD:R_0603_1608Metric_Pad0.98x0.95mm_HandSolder, F.Cu at (36.4, 57.6)
- added Rc9: R, Resistor_SMD:R_0603_1608Metric_Pad0.98x0.95mm_HandSolder, F.Cu at (36.4, 60.1)
- added Rl1: R, Resistor_SMD:R_0603_1608Metric_Pad0.98x0.95mm_HandSolder, F.Cu at (45.1, 60.1)
- added Rl10: R, Resistor_SMD:R_0603_1608Metric_Pad0.98x0.95mm_HandSolder, F.Cu at (49.4, 52.6)
- added Rl11: R, Resistor_SMD:R_0603_1608Metric_Pad0.98x0.95mm_HandSolder, F.Cu at (49.4, 55.1)
- added Rl12: R, Resistor_SMD:R_0603_1608Metric_Pad0.98x0.95mm_HandSolder, F.Cu at (49.4, 57.6)
- added Rl13: R, Resistor_SMD:R_0603_1608Metric_Pad0.98x0.95mm_HandSolder, F.Cu at (49.4, 60.1)
- added Rl14: R, Resistor_SMD:R_0603_1608Metric_Pad0.98x0.95mm_HandSolder, F.Cu at (49.4, 62.6)
- added Rl15: R, Resistor_SMD:R_0603_1608Metric_Pad0.98x0.95mm_HandSolder, F.Cu at (49.4, 65.1)
- added Rl16: R, Resistor_SMD:R_0603_1608Metric_Pad0.98x0.95mm_HandSolder, F.Cu at (49.4, 67.7)
- added Rl17: R, Resistor_SMD:R_0603_1608Metric_Pad0.98x0.95mm_HandSolder, F.Cu at (49.4, 70.2)
- added Rl18: R, Resistor_SMD:R_0603_1608Metric_Pad0.98x0.95mm_HandSolder, F.Cu at (49.4, 72.7)
- added Rl19: R, Resistor_SMD:R_0603_1608Metric_Pad0.98x0.95mm_HandSolder, F.Cu at (53.8, 45.1)
- added Rl2: R, Resistor_SMD:R_0603_1608Metric_Pad0.98x0.95mm_HandSolder, F.Cu at (45.1, 62.6)
- added Rl20: R, Resistor_SMD:R_0603_1608Metric_Pad0.98x0.95mm_HandSolder, F.Cu at (53.8, 47.6)
- added Rl21: R, Resistor_SMD:R_0603_1608Metric_Pad0.98x0.95mm_HandSolder, F.Cu at (53.8, 50.1)
- added Rl22: R, Resistor_SMD:R_0603_1608Metric_Pad0.98x0.95mm_HandSolder, F.Cu at (53.8, 52.6)
- added Rl23: R, Resistor_SMD:R_0603_1608Metric_Pad0.98x0.95mm_HandSolder, F.Cu at (53.8, 55.1)
- added Rl24: R, Resistor_SMD:R_0603_1608Metric_Pad0.98x0.95mm_HandSolder, F.Cu at (53.8, 57.6)
- added Rl25: R, Resistor_SMD:R_0603_1608Metric_Pad0.98x0.95mm_HandSolder, F.Cu at (53.8, 60.1)
- added Rl26: R, Resistor_SMD:R_0603_1608Metric_Pad0.98x0.95mm_HandSolder, F.Cu at (53.8, 62.6)
- added Rl27: R, Resistor_SMD:R_0603_1608Metric_Pad0.98x0.95mm_HandSolder, F.Cu at (53.8, 65.1)
- added Rl28: R, Resistor_SMD:R_0603_1608Metric_Pad0.98x0.95mm_HandSolder, F.Cu at (53.8, 67.7)
- added Rl29: R, Resistor_SMD:R_0603_1608Metric_Pad0.98x0.95mm_HandSolder, F.Cu at (53.8, 70.2)
- added Rl3: R, Resistor_SMD:R_0603_1608Metric_Pad0.98x0.95mm_HandSolder, F.Cu at (45.1, 65.1)
- added Rl30: R, Resistor_SMD:R_0603_1608Metric_Pad0.98x0.95mm_HandSolder, F.Cu at (53.8, 72.7)
- added Rl31: R, Resistor_SMD:R_0603_1608Metric_Pad0.98x0.95mm_HandSolder, F.Cu at (58.1, 45.1)
- added Rl32: R, Resistor_SMD:R_0603_1608Metric_Pad0.98x0.95mm_HandSolder, F.Cu at (58.1, 47.6)
- added Rl4: R, Resistor_SMD:R_0603_1608Metric_Pad0.98x0.95mm_HandSolder, F.Cu at (45.1, 67.7)
- added Rl5: R, Resistor_SMD:R_0603_1608Metric_Pad0.98x0.95mm_HandSolder, F.Cu at (45.1, 70.2)
- added Rl6: R, Resistor_SMD:R_0603_1608Metric_Pad0.98x0.95mm_HandSolder, F.Cu at (45.1, 72.7)
- added Rl7: R, Resistor_SMD:R_0603_1608Metric_Pad0.98x0.95mm_HandSolder, F.Cu at (49.4, 45.1)
- added Rl8: R, Resistor_SMD:R_0603_1608Metric_Pad0.98x0.95mm_HandSolder, F.Cu at (49.4, 47.6)
- added Rl9: R, Resistor_SMD:R_0603_1608Metric_Pad0.98x0.95mm_HandSolder, F.Cu at (49.4, 50.1)
- added Rs1: R, Resistor_SMD:R_0603_1608Metric_Pad0.98x0.95mm_HandSolder, F.Cu at (58.1, 50.1)
- added Rs10: R, Resistor_SMD:R_0603_1608Metric_Pad0.98x0.95mm_HandSolder, F.Cu at (58.1, 72.7)
- added Rs11: R, Resistor_SMD:R_0603_1608Metric_Pad0.98x0.95mm_HandSolder, F.Cu at (62.5, 45.1)
- added Rs12: R, Resistor_SMD:R_0603_1608Metric_Pad0.98x0.95mm_HandSolder, F.Cu at (62.5, 47.6)
- added Rs13: R, Resistor_SMD:R_0603_1608Metric_Pad0.98x0.95mm_HandSolder, F.Cu at (62.5, 50.1)
- added Rs14: R, Resistor_SMD:R_0603_1608Metric_Pad0.98x0.95mm_HandSolder, F.Cu at (62.5, 52.6)
- added Rs15: R, Resistor_SMD:R_0603_1608Metric_Pad0.98x0.95mm_HandSolder, F.Cu at (62.5, 55.1)
- added Rs16: R, Resistor_SMD:R_0603_1608Metric_Pad0.98x0.95mm_HandSolder, F.Cu at (62.5, 57.6)
- added Rs17: R, Resistor_SMD:R_0603_1608Metric_Pad0.98x0.95mm_HandSolder, F.Cu at (62.5, 60.1)
- added Rs18: R, Resistor_SMD:R_0603_1608Metric_Pad0.98x0.95mm_HandSolder, F.Cu at (62.5, 62.6)
- added Rs19: R, Resistor_SMD:R_0603_1608Metric_Pad0.98x0.95mm_HandSolder, F.Cu at (62.5, 65.1)
- added Rs2: R, Resistor_SMD:R_0603_1608Metric_Pad0.98x0.95mm_HandSolder, F.Cu at (58.1, 52.6)
- added Rs20: R, Resistor_SMD:R_0603_1608Metric_Pad0.98x0.95mm_HandSolder, F.Cu at (62.5, 67.7)
- added Rs21: R, Resistor_SMD:R_0603_1608Metric_Pad0.98x0.95mm_HandSolder, F.Cu at (62.5, 70.2)
- added Rs22: R, Resistor_SMD:R_0603_1608Metric_Pad0.98x0.95mm_HandSolder, F.Cu at (62.5, 72.7)
- added Rs23: R, Resistor_SMD:R_0603_1608Metric_Pad0.98x0.95mm_HandSolder, F.Cu at (66.8, 45.1)
- added Rs24: R, Resistor_SMD:R_0603_1608Metric_Pad0.98x0.95mm_HandSolder, F.Cu at (66.8, 47.6)
- added Rs25: R, Resistor_SMD:R_0603_1608Metric_Pad0.98x0.95mm_HandSolder, F.Cu at (66.8, 50.1)
- added Rs26: R, Resistor_SMD:R_0603_1608Metric_Pad0.98x0.95mm_HandSolder, F.Cu at (66.8, 52.6)
- added Rs27: R, Resistor_SMD:R_0603_1608Metric_Pad0.98x0.95mm_HandSolder, F.Cu at (66.8, 55.1)
- added Rs28: R, Resistor_SMD:R_0603_1608Metric_Pad0.98x0.95mm_HandSolder, F.Cu at (66.8, 57.6)
- added Rs29: R, Resistor_SMD:R_0603_1608Metric_Pad0.98x0.95mm_HandSolder, F.Cu at (66.8, 60.1)
- added Rs3: R, Resistor_SMD:R_0603_1608Metric_Pad0.98x0.95mm_HandSolder, F.Cu at (58.1, 55.1)
- added Rs30: R, Resistor_SMD:R_0603_1608Metric_Pad0.98x0.95mm_HandSolder, F.Cu at (66.8, 62.6)
- added Rs31: R, Resistor_SMD:R_0603_1608Metric_Pad0.98x0.95mm_HandSolder, F.Cu at (66.8, 65.1)
- added Rs32: R, Resistor_SMD:R_0603_1608Metric_Pad0.98x0.95mm_HandSolder, F.Cu at (66.8, 67.7)
- added Rs4: R, Resistor_SMD:R_0603_1608Metric_Pad0.98x0.95mm_HandSolder, F.Cu at (58.1, 57.6)
- added Rs5: R, Resistor_SMD:R_0603_1608Metric_Pad0.98x0.95mm_HandSolder, F.Cu at (58.1, 60.1)
- added Rs6: R, Resistor_SMD:R_0603_1608Metric_Pad0.98x0.95mm_HandSolder, F.Cu at (58.1, 62.6)
- added Rs7: R, Resistor_SMD:R_0603_1608Metric_Pad0.98x0.95mm_HandSolder, F.Cu at (58.1, 65.1)
- added Rs8: R, Resistor_SMD:R_0603_1608Metric_Pad0.98x0.95mm_HandSolder, F.Cu at (58.1, 67.7)
- added Rs9: R, Resistor_SMD:R_0603_1608Metric_Pad0.98x0.95mm_HandSolder, F.Cu at (58.1, 70.2)
- added U1: LM339, Package_SO:SOIC-14_3.9x8.7mm_P1.27mm, F.Cu at (80.3, 79.2)
- added U2: LM339, Package_SO:SOIC-14_3.9x8.7mm_P1.27mm, F.Cu at (88.8, 79.2)
- added U3: LM339, Package_SO:SOIC-14_3.9x8.7mm_P1.27mm, F.Cu at (71.9, 89.6)
- added U4: LM339, Package_SO:SOIC-14_3.9x8.7mm_P1.27mm, F.Cu at (80.3, 89.6)
- added U5: LM339, Package_SO:SOIC-14_3.9x8.7mm_P1.27mm, F.Cu at (88.8, 89.6)
- added U6: LM339, Package_SO:SOIC-14_3.9x8.7mm_P1.27mm, F.Cu at (71.9, 99.9)
- added U7: LM339, Package_SO:SOIC-14_3.9x8.7mm_P1.27mm, F.Cu at (80.3, 99.9)
- added U8: LM339, Package_SO:SOIC-14_3.9x8.7mm_P1.27mm, F.Cu at (88.8, 99.9)
- Q1: footprint ALS-PT19-315C:ALS-PT19-315C -> hankotei:hankotei_node
- moved Q1 27.8 mm to (97.5, 97.6)
Connections:
- Q1 pad 1: unconnected-(Q1-C-Pad1) -> VCC
- Q1 pad 2: unconnected-(Q1-E-Pad2) -> Net-(Q1-E)
Other:
- board outline added: 116.6 x 113 mm
