File: KiCad/prot2/基盤外形までバックアップ/prot2/prot2.kicad_pcb (KiCad board)
At the start: 2 copper layers, 140 x 140 mm, 193 parts, among them J1 Conn_01x02_Socket, J2 LED_SW, J3 Conn_01x04_Socket, Q1 Q_Photo_NPN, U1 LM339, U2 LM339, U3 LM339, U4 LM339, U5 LM339, U6 LM339, U7 LM339, U8 LM339

Commit message: 外形まで完成くそ
Parts:
- removed the Rl1 at (539.6, 551.6)
- removed the Rl1 at (561.6, 520.9)
- removed the Rl1 at (448.4, 539.6)
- removed the Rl1 at (495.7, 435.1)
- removed the Rl1 at (558.3, 471.3)
- removed the Rl1 at (479.1, 561.6)
- removed the Rl1 at (562.8, 483.2)
- removed the Rl1 at (508.5, 435.6)
- removed the Rl1 at (491.5, 564.4)
- removed the Rl1 at (443.7, 467.5)
- removed the Rl1 at (437.2, 516.8)
- removed the Rl1 at (504.3, 564.9)
- removed the Rl1 at (532.5, 443.7)
- removed the Rl1 at (520.9, 438.4)
- removed the Rl1 at (528.7, 558.3)
- removed the Rl1 at (471.3, 441.7)
- removed the Rl1 at (551.6, 460.4)
- removed the Rl1 at (451.1, 457.1)
- removed the Rl1 at (441.7, 528.7)
- removed the Rl1 at (542.9, 451.1)
- removed the Rl1 at (467.5, 556.3)
- removed the Rl1 at (556.3, 532.5)
- removed the Rl1 at (457.1, 548.9)
- removed the Rl1 at (516.8, 562.8)
- removed the Rl1 at (564.9, 495.7)
- removed the Rl1 at (435.1, 504.3)
- removed the Rl1 at (548.9, 542.9)
- removed the Rl1 at (438.4, 479.1)
- removed the Rl1 at (483.2, 437.2)
- removed the Rl1 at (435.6, 491.5)
- removed the Rl1 at (460.4, 448.4)
- removed the Rs1 at (458.6, 553.9)
- removed the Rs1 at (530.1, 439.0)
- removed the Rs1 at (482.4, 565.7)
- removed the Rs1 at (558.9, 466.0)
- removed the Rs1 at (446.1, 458.6)
- removed the Rs1 at (567.9, 504.4)
- removed the Rs1 at (567.4, 491.1)
- removed the Rs1 at (466.0, 441.1)
- removed the Rs1 at (534.0, 558.9)
- removed the Rs1 at (435.6, 521.9)
- removed the Rs1 at (495.6, 567.9)
- removed the Rs1 at (504.4, 432.1)
- removed the Rs1 at (508.9, 567.4)
- removed the Rs1 at (521.9, 564.4)
- removed the Rs1 at (553.9, 541.4)
- removed the Rs1 at (469.9, 561.0)
- removed the Rs1 at (561.0, 530.1)
- removed the Rs1 at (564.4, 478.1)
- removed the Rs1 at (455.2, 448.9)
- removed the Rs1 at (551.1, 455.2)
- removed the Rs1 at (448.9, 544.8)
- removed the Rs1 at (544.8, 551.1)
- removed the Rs1 at (517.6, 434.3)
- removed the Rs1 at (541.4, 446.1)
- removed the Rs1 at (434.3, 482.4)
- removed the Rs1 at (432.1, 495.6)
- removed the Rs1 at (432.6, 508.9)
- removed the Rs1 at (441.1, 534.0)
- removed the Rs1 at (491.1, 432.6)
- removed the Rs1 at (439.0, 469.9)
- removed the Rs1 at (478.1, 435.6)
- added Rl10: R, Resistor_SMD:R_0603_1608Metric_Pad0.98x0.95mm_HandSolder, F.Cu at (325.0, 476.2)
- added Rl11: R, Resistor_SMD:R_0603_1608Metric_Pad0.98x0.95mm_HandSolder, F.Cu at (325.0, 478.7)
- added Rl12: R, Resistor_SMD:R_0603_1608Metric_Pad0.98x0.95mm_HandSolder, F.Cu at (325.0, 481.2)
- added Rl13: R, Resistor_SMD:R_0603_1608Metric_Pad0.98x0.95mm_HandSolder, F.Cu at (325.0, 483.7)
- added Rl14: R, Resistor_SMD:R_0603_1608Metric_Pad0.98x0.95mm_HandSolder, F.Cu at (325.0, 486.2)
- added Rl15: R, Resistor_SMD:R_0603_1608Metric_Pad0.98x0.95mm_HandSolder, F.Cu at (325.0, 488.7)
- added Rl16: R, Resistor_SMD:R_0603_1608Metric_Pad0.98x0.95mm_HandSolder, F.Cu at (325.0, 491.2)
- added Rl17: R, Resistor_SMD:R_0603_1608Metric_Pad0.98x0.95mm_HandSolder, F.Cu at (325.0, 493.8)
- added Rl18: R, Resistor_SMD:R_0603_1608Metric_Pad0.98x0.95mm_HandSolder, F.Cu at (325.0, 496.3)
- added Rl19: R, Resistor_SMD:R_0603_1608Metric_Pad0.98x0.95mm_HandSolder, F.Cu at (329.4, 468.7)
- added Rl2: R, Resistor_SMD:R_0603_1608Metric_Pad0.98x0.95mm_HandSolder, F.Cu at (320.7, 486.2)
- added Rl20: R, Resistor_SMD:R_0603_1608Metric_Pad0.98x0.95mm_HandSolder, F.Cu at (329.4, 471.2)
- added Rl21: R, Resistor_SMD:R_0603_1608Metric_Pad0.98x0.95mm_HandSolder, F.Cu at (329.4, 473.7)
- added Rl22: R, Resistor_SMD:R_0603_1608Metric_Pad0.98x0.95mm_HandSolder, F.Cu at (329.4, 476.2)
- added Rl23: R, Resistor_SMD:R_0603_1608Metric_Pad0.98x0.95mm_HandSolder, F.Cu at (329.4, 478.7)
- added Rl24: R, Resistor_SMD:R_0603_1608Metric_Pad0.98x0.95mm_HandSolder, F.Cu at (329.4, 481.2)
- added Rl25: R, Resistor_SMD:R_0603_1608Metric_Pad0.98x0.95mm_HandSolder, F.Cu at (329.4, 483.7)
- added Rl26: R, Resistor_SMD:R_0603_1608Metric_Pad0.98x0.95mm_HandSolder, F.Cu at (329.4, 486.2)
- added Rl27: R, Resistor_SMD:R_0603_1608Metric_Pad0.98x0.95mm_HandSolder, F.Cu at (329.4, 488.7)
- added Rl28: R, Resistor_SMD:R_0603_1608Metric_Pad0.98x0.95mm_HandSolder, F.Cu at (329.4, 491.2)
- added Rl29: R, Resistor_SMD:R_0603_1608Metric_Pad0.98x0.95mm_HandSolder, F.Cu at (329.4, 493.8)
- added Rl3: R, Resistor_SMD:R_0603_1608Metric_Pad0.98x0.95mm_HandSolder, F.Cu at (320.7, 488.7)
- added Rl30: R, Resistor_SMD:R_0603_1608Metric_Pad0.98x0.95mm_HandSolder, F.Cu at (329.4, 496.3)
- added Rl31: R, Resistor_SMD:R_0603_1608Metric_Pad0.98x0.95mm_HandSolder, F.Cu at (333.7, 468.7)
- added Rl32: R, Resistor_SMD:R_0603_1608Metric_Pad0.98x0.95mm_HandSolder, F.Cu at (333.7, 471.2)
- added Rl4: R, Resistor_SMD:R_0603_1608Metric_Pad0.98x0.95mm_HandSolder, F.Cu at (320.7, 491.2)
- added Rl5: R, Resistor_SMD:R_0603_1608Metric_Pad0.98x0.95mm_HandSolder, F.Cu at (320.7, 493.8)
- added Rl6: R, Resistor_SMD:R_0603_1608Metric_Pad0.98x0.95mm_HandSolder, F.Cu at (320.7, 496.3)
- added Rl7: R, Resistor_SMD:R_0603_1608Metric_Pad0.98x0.95mm_HandSolder, F.Cu at (325.0, 468.7)
- added Rl8: R, Resistor_SMD:R_0603_1608Metric_Pad0.98x0.95mm_HandSolder, F.Cu at (325.0, 471.2)
- added Rl9: R, Resistor_SMD:R_0603_1608Metric_Pad0.98x0.95mm_HandSolder, F.Cu at (325.0, 473.7)
- added Rs10: R, Resistor_SMD:R_0603_1608Metric_Pad0.98x0.95mm_HandSolder, F.Cu at (333.7, 496.3)
- added Rs11: R, Resistor_SMD:R_0603_1608Metric_Pad0.98x0.95mm_HandSolder, F.Cu at (338.1, 468.7)
- added Rs12: R, Resistor_SMD:R_0603_1608Metric_Pad0.98x0.95mm_HandSolder, F.Cu at (338.1, 471.2)
- added Rs13: R, Resistor_SMD:R_0603_1608Metric_Pad0.98x0.95mm_HandSolder, F.Cu at (338.1, 473.7)
- added Rs14: R, Resistor_SMD:R_0603_1608Metric_Pad0.98x0.95mm_HandSolder, F.Cu at (338.1, 476.2)
- added Rs15: R, Resistor_SMD:R_0603_1608Metric_Pad0.98x0.95mm_HandSolder, F.Cu at (338.1, 478.7)
- added Rs16: R, Resistor_SMD:R_0603_1608Metric_Pad0.98x0.95mm_HandSolder, F.Cu at (338.1, 481.2)
- added Rs17: R, Resistor_SMD:R_0603_1608Metric_Pad0.98x0.95mm_HandSolder, F.Cu at (338.1, 483.7)
- added Rs18: R, Resistor_SMD:R_0603_1608Metric_Pad0.98x0.95mm_HandSolder, F.Cu at (338.1, 486.2)
- added Rs19: R, Resistor_SMD:R_0603_1608Metric_Pad0.98x0.95mm_HandSolder, F.Cu at (338.1, 488.7)
- added Rs2: R, Resistor_SMD:R_0603_1608Metric_Pad0.98x0.95mm_HandSolder, F.Cu at (505.0, 482.4)
- added Rs20: R, Resistor_SMD:R_0603_1608Metric_Pad0.98x0.95mm_HandSolder, F.Cu at (338.1, 491.2)
- added Rs21: R, Resistor_SMD:R_0603_1608Metric_Pad0.98x0.95mm_HandSolder, F.Cu at (338.1, 493.8)
- added Rs22: R, Resistor_SMD:R_0603_1608Metric_Pad0.98x0.95mm_HandSolder, F.Cu at (338.1, 496.3)
- added Rs23: R, Resistor_SMD:R_0603_1608Metric_Pad0.98x0.95mm_HandSolder, F.Cu at (342.4, 468.7)
- added Rs24: R, Resistor_SMD:R_0603_1608Metric_Pad0.98x0.95mm_HandSolder, F.Cu at (342.4, 471.2)
- added Rs25: R, Resistor_SMD:R_0603_1608Metric_Pad0.98x0.95mm_HandSolder, F.Cu at (342.4, 473.7)
- added Rs26: R, Resistor_SMD:R_0603_1608Metric_Pad0.98x0.95mm_HandSolder, F.Cu at (342.4, 476.2)
- added Rs27: R, Resistor_SMD:R_0603_1608Metric_Pad0.98x0.95mm_HandSolder, F.Cu at (342.4, 478.7)
- added Rs28: R, Resistor_SMD:R_0603_1608Metric_Pad0.98x0.95mm_HandSolder, F.Cu at (342.4, 481.2)
- added Rs29: R, Resistor_SMD:R_0603_1608Metric_Pad0.98x0.95mm_HandSolder, F.Cu at (342.4, 483.7)
- added Rs3: R, Resistor_SMD:R_0603_1608Metric_Pad0.98x0.95mm_HandSolder, F.Cu at (505.0, 484.9)
- added Rs30: R, Resistor_SMD:R_0603_1608Metric_Pad0.98x0.95mm_HandSolder, F.Cu at (342.4, 486.2)
- added Rs31: R, Resistor_SMD:R_0603_1608Metric_Pad0.98x0.95mm_HandSolder, F.Cu at (342.4, 488.7)
- added Rs32: R, Resistor_SMD:R_0603_1608Metric_Pad0.98x0.95mm_HandSolder, F.Cu at (342.4, 491.2)
- added Rs4: R, Resistor_SMD:R_0603_1608Metric_Pad0.98x0.95mm_HandSolder, F.Cu at (505.0, 487.4)
- added Rs5: R, Resistor_SMD:R_0603_1608Metric_Pad0.98x0.95mm_HandSolder, F.Cu at (333.7, 483.7)
- added Rs6: R, Resistor_SMD:R_0603_1608Metric_Pad0.98x0.95mm_HandSolder, F.Cu at (333.7, 486.2)
- added Rs7: R, Resistor_SMD:R_0603_1608Metric_Pad0.98x0.95mm_HandSolder, F.Cu at (333.7, 488.7)
- added Rs8: R, Resistor_SMD:R_0603_1608Metric_Pad0.98x0.95mm_HandSolder, F.Cu at (333.7, 491.2)
- added Rs9: R, Resistor_SMD:R_0603_1608Metric_Pad0.98x0.95mm_HandSolder, F.Cu at (333.7, 493.8)
- moved Rl1 245.0 mm to (320.7, 483.7), turned to 0 degrees
- moved Rc1 81.3 mm to (478.9, 500.0), turned to 0 degrees
- moved Rc2 77.1 mm to (478.9, 502.5), turned to 0 degrees
- moved Rc4 72.6 mm to (483.2, 477.4), turned to 0 degrees
- moved Rc3 70.8 mm to (483.2, 474.9), turned to 0 degrees
- moved U1 41.8 mm to (527.1, 509.0), turned to 0 degrees
- moved Rs1 15.1 mm to (558.3, 504.4), turned to -90 degrees
- renumbered D1 to D10, D1 to D11, D1 to D12, D1 to D13, D1 to D14, D1 to D15, D1 to D16, D1 to D17, D1 to D18, D1 to D19, D1 to D2, D1 to D20, D1 to D21, D1 to D22, D1 to D23, D1 to D24, D1 to D25, D1 to D26, D1 to D27, D1 to D28, D1 to D29, D1 to D3, D1 to D30, D1 to D31, D1 to D32, D1 to D4, D1 to D5, D1 to D6, D1 to D7, D1 to D8, D1 to D9, Q1 to Q10, Q1 to Q11, Q1 to Q12, Q1 to Q13, Q1 to Q14, Q1 to Q15, Q1 to Q16, Q1 to Q17, Q1 to Q18, Q1 to Q19, Q1 to Q2, Q1 to Q20, Q1 to Q21, Q1 to Q22, Q1 to Q23, Q1 to Q24, Q1 to Q25, Q1 to Q26, Q1 to Q27, Q1 to Q28, Q1 to Q29, Q1 to Q3, Q1 to Q30, Q1 to Q31, Q1 to Q32, Q1 to Q4, Q1 to Q5, Q1 to Q6, Q1 to Q7, Q1 to Q8, Q1 to Q9
Connections:
- RP2040_Zero2 pad 1: 4 -> unconnected-(RP2040_Zero2-0-Pad1)
- RP2040_Zero2 pad 2: 3 -> unconnected-(RP2040_Zero2-1-Pad2)
- RP2040_Zero2 pad 3: 2 -> unconnected-(RP2040_Zero2-2-Pad3)
- RP2040_Zero2 pad 4: 1 -> unconnected-(RP2040_Zero2-3-Pad4)
Routing:
- net Net-(Q1-E): track 86.0 -> 0.00 mm
- net Net-(D1-K): track 79.0 -> 0.00 mm
- net VCC: track 4.28 -> 0.00 mm
- net GND: track 1.44 -> 0.00 mm, vias 1 -> 0
