File: KiCad/prot3/prot3.kicad_pcb (KiCad board)
At the start: 2 copper layers, 140 x 140 mm, 193 parts, among them J1 Conn_01x02_Socket, J2 LED_SW, J3 Conn_01x04_Socket, Q1 Q_Photo_NPN, Q10 Q_Photo_NPN, Q11 Q_Photo_NPN, Q12 Q_Photo_NPN, Q13 Q_Photo_NPN, Q14 Q_Photo_NPN, Q15 Q_Photo_NPN, Q16 Q_Photo_NPN, Q17 Q_Photo_NPN, Q18 Q_Photo_NPN, Q19 Q_Photo_NPN, Q2 Q_Photo_NPN, Q20 Q_Photo_NPN, Q21 Q_Photo_NPN, Q22 Q_Photo_NPN, Q23 Q_Photo_NPN, Q24 Q_Photo_NPN, Q25 Q_Photo_NPN, Q26 Q_Photo_NPN, Q27 Q_Photo_NPN, Q28 Q_Photo_NPN, Q29 Q_Photo_NPN, Q3 Q_Photo_NPN, Q30 Q_Photo_NPN, Q31 Q_Photo_NPN, Q32 Q_Photo_NPN, Q4 Q_Photo_NPN, Q5 Q_Photo_NPN, Q6 Q_Photo_NPN, Q7 Q_Photo_NPN, Q8 Q_Photo_NPN, Q9 Q_Photo_NPN, U1 LM339, U2 LM339, U3 LM339, U4 LM339, U5 LM339, U6 LM339, U7 LM339, U8 LM339

Commit message: RP2040_kimoi1
Parts:
- added B1: R, Resistor_SMD:R_0603_1608Metric_Pad0.98x0.95mm_HandSolder, F.Cu at (354.1, 484.2)
- added B2: R, Resistor_SMD:R_0603_1608Metric_Pad0.98x0.95mm_HandSolder, F.Cu at (354.1, 486.7)
- added C14: C, Capacitor_SMD:C_0603_1608Metric_Pad1.08x0.95mm_HandSolder, F.Cu at (354.1, 489.2)
- added C15: C, Capacitor_SMD:C_0603_1608Metric_Pad1.08x0.95mm_HandSolder, F.Cu at (354.1, 491.7)
- added R1: R, Resistor_SMD:R_0603_1608Metric_Pad0.98x0.95mm_HandSolder, F.Cu at (354.1, 494.2)
- C11: footprint Package_SO:SOIC-14_3.9x8.7mm_P1.27mm -> Capacitor_THT:C_Radial_D8.0mm_H11.5mm_P3.50mm
- RP2040_Zero1: footprint RP2040zero:RP2040_zero -> RP2040_zero_kimoi1:RP2040_zero_kimoi2
- RP2040_Zero2: footprint RP2040zero:RP2040_zero -> RP2040_zero_kimoi1:RP2040_zero_kimoi1
- moved RP2040_Zero2 197.2 mm to (529.5, 524.5), turned to 90 degrees
- moved U8 188.1 mm to (551.7, 507.0)
- moved U2 166.6 mm to (527.0, 467.1)
- moved U7 162.4 mm to (515.8, 551.5)
- moved RP2040_Zero1 158.8 mm to (471.6, 525.7), turned to -90 degrees
- moved U3 138.5 mm to (476.4, 462.7)
- moved U6 132.5 mm to (477.4, 549.4)
- moved U4 114.0 mm to (461.6, 470.6)
- moved U5 80.7 mm to (444.0, 500.2)
- moved Rc4 0.07 mm to (548.9, 479.4)
Connections:
- RV1 pad 2: conp_+ -> Net-(B2-Pad1)
Other:
- board text added: "5v"
