File: KiCad/prot3/prot3.kicad_sch (KiCad schematic)
At the start: 193 parts, among them J1 Conn_01x02_Socket, J2 LED_SW, J3 Conn_01x04_Socket, Q1 Q_Photo_NPN, Q10 Q_Photo_NPN, Q11 Q_Photo_NPN, Q12 Q_Photo_NPN, Q13 Q_Photo_NPN, Q14 Q_Photo_NPN, Q15 Q_Photo_NPN, Q16 Q_Photo_NPN, Q17 Q_Photo_NPN, Q18 Q_Photo_NPN, Q19 Q_Photo_NPN, Q2 Q_Photo_NPN, Q20 Q_Photo_NPN, Q21 Q_Photo_NPN, Q22 Q_Photo_NPN, Q23 Q_Photo_NPN, Q24 Q_Photo_NPN, Q25 Q_Photo_NPN, Q26 Q_Photo_NPN, Q27 Q_Photo_NPN, Q28 Q_Photo_NPN, Q29 Q_Photo_NPN, Q3 Q_Photo_NPN, Q30 Q_Photo_NPN, Q31 Q_Photo_NPN, Q32 Q_Photo_NPN, Q4 Q_Photo_NPN, Q5 Q_Photo_NPN, Q6 Q_Photo_NPN, Q7 Q_Photo_NPN, Q8 Q_Photo_NPN, Q9 Q_Photo_NPN, U1 LM339, U2 LM339, U3 LM339, U4 LM339, U5 LM339, U6 LM339, U7 LM339, U8 LM339

Commit message: PWMしきい値回路
Parts:
- added B1, B2, R1: R, Resistor_SMD:R_0603_1608Metric_Pad0.98x0.95mm_HandSolder, symbol Device:R
- added C14, C15: C, Capacitor_SMD:C_0603_1608Metric_Pad1.08x0.95mm_HandSolder, symbol Device:C
Connections:
- net GND: now also C15.2
- net VCC: now also C14.1
- net conp_+: now also B1.2, B2.2; no longer RV1.2
- new net: B1.1, C14.2, C15.1, R1.2
- new net: B2.1, RV1.2
- new net Conp_PWM: R1.1
Other:
- note added: "10nF"
- note added: "Bridge"
- note added: "とりあえず10ｋΩ1608"
- moved on the sheet: RV1

Commit message: RP2040_kimoi1
Parts:
- C11: footprint Package_SO:SOIC-14_3.9x8.7mm_P1.27mm -> Capacitor_THT:C_Radial_D8.0mm_H11.5mm_P3.50mm
- RP2040_Zero1: footprint RP2040zero:RP2040_zero -> RP2040_zero_kimoi1:RP2040_zero_kimoi2
- RP2040_Zero2: footprint RP2040zero:RP2040_zero -> RP2040_zero_kimoi1:RP2040_zero_kimoi1
Changed lines of the file:
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@@
 			)
 		)
-		(property "Footprint" "Package_SO:SOIC-14_3.9x8.7mm_P1.27mm"
+		(property "Footprint" "Capacitor_THT:C_Radial_D8.0mm_H11.5mm_P3.50mm"
 			(at 63.5 276.86 0)
 			(effects
@@
 			)
 		)
-		(property "Footprint" "RP2040zero:RP2040_zero"
+		(property "Footprint" "RP2040_zero_kimoi1:RP2040_zero_kimoi2"
 			(at 100.33 287.02 0)
 			(effects
@@
 			)
 		)
-		(property "Footprint" "RP2040zero:RP2040_zero"
+		(property "Footprint" "RP2040_zero_kimoi1:RP2040_zero_kimoi1"
 			(at 194.31 289.56 0)
 			(effects
