File: KiCad/prot3/8.1バックアップ1/prot3.kicad_pcb (KiCad board)
At the start: 2 copper layers, 140 x 140 mm, 198 parts, among them J1 Conn_01x02_Socket, J2 LED_SW, J3 Conn_01x04_Socket, Q1 Q_Photo_NPN, Q10 Q_Photo_NPN, Q11 Q_Photo_NPN, Q12 Q_Photo_NPN, Q13 Q_Photo_NPN, Q14 Q_Photo_NPN, Q15 Q_Photo_NPN, Q16 Q_Photo_NPN, Q17 Q_Photo_NPN, Q18 Q_Photo_NPN, Q19 Q_Photo_NPN, Q2 Q_Photo_NPN, Q20 Q_Photo_NPN, Q21 Q_Photo_NPN, Q22 Q_Photo_NPN, Q23 Q_Photo_NPN, Q24 Q_Photo_NPN, Q25 Q_Photo_NPN, Q26 Q_Photo_NPN, Q27 Q_Photo_NPN, Q28 Q_Photo_NPN, Q29 Q_Photo_NPN, Q3 Q_Photo_NPN, Q30 Q_Photo_NPN, Q31 Q_Photo_NPN, Q32 Q_Photo_NPN, Q4 Q_Photo_NPN, Q5 Q_Photo_NPN, Q6 Q_Photo_NPN, Q7 Q_Photo_NPN, Q8 Q_Photo_NPN, Q9 Q_Photo_NPN, U1 LM339, U2 LM339, U3 LM339, U4 LM339, U5 LM339, U6 LM339, U7 LM339, U8 LM339

Commit message: コンパレーターchに名札配置、rpzero仮完成
Parts:
- J1, J3: moved to F.Cu
- moved C10 216.8 mm to (307.6, 491.2)
- moved Rc13 200.2 mm to (312.0, 493.8)
- moved Rc14 200.2 mm to (312.0, 496.3)
- moved C3 199.7 mm to (307.6, 473.7)
- moved Rc15 197.2 mm to (316.3, 468.7)
- moved Rc16 197.2 mm to (316.3, 471.2)
- moved Rc10 196.4 mm to (312.0, 486.2)
- moved Rc11 196.4 mm to (312.0, 488.7)
- moved Rc12 196.4 mm to (312.0, 491.2)
- moved Rc9 196.4 mm to (312.0, 483.7)
- moved Rc5 196.3 mm to (312.0, 473.7)
- moved Rc6 196.3 mm to (312.0, 476.2)
- moved Rc7 196.3 mm to (312.0, 478.7)
- moved Rc8 196.3 mm to (312.0, 481.2)
- moved C4 192.1 mm to (307.6, 476.2)
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Connections:
- C1 pad 2: LED_5V -> GND
- C10 pad 2: LED_5V -> GND
- C11 pad 2: LED_5V -> GND
- C12 pad 2: LED_5V -> GND
- C13 pad 2: LED_5V -> GND
- C15 pad 2: LED_5V -> GND
- C2 pad 2: LED_5V -> GND
- C3 pad 2: LED_5V -> GND
- C4 pad 2: LED_5V -> GND
- C5 pad 2: LED_5V -> GND
- C6 pad 2: LED_5V -> GND
- C7 pad 2: LED_5V -> GND
- C8 pad 2: LED_5V -> GND
- C9 pad 2: LED_5V -> GND
- J1 pad 2: LED_5V -> GND
- J3 pad 4: LED_5V -> GND
- RP2040_Zero1 pad 22: LED_5V -> GND
- RP2040_Zero2 pad 22: LED_5V -> GND
- RV1 pad 3: LED_5V -> GND
- Rl1 pad 2: LED_5V -> GND
- Rl10 pad 2: LED_5V -> GND
- Rl11 pad 2: LED_5V -> GND
- Rl12 pad 2: LED_5V -> GND
- Rl13 pad 2: LED_5V -> GND
- Rl14 pad 2: LED_5V -> GND
- Rl15 pad 2: LED_5V -> GND
- Rl16 pad 2: LED_5V -> GND
- Rl17 pad 2: LED_5V -> GND
- Rl18 pad 2: LED_5V -> GND
- Rl19 pad 2: LED_5V -> GND
- Rl2 pad 2: LED_5V -> GND
- Rl20 pad 2: LED_5V -> GND
- Rl21 pad 2: LED_5V -> GND
- Rl22 pad 2: LED_5V -> GND
- Rl23 pad 2: LED_5V -> GND
- Rl24 pad 2: LED_5V -> GND
- Rl25 pad 2: LED_5V -> GND
- Rl26 pad 2: LED_5V -> GND
- Rl27 pad 2: LED_5V -> GND
- Rl28 pad 2: LED_5V -> GND
- Rl29 pad 2: LED_5V -> GND
- Rl3 pad 2: LED_5V -> GND
- Rl30 pad 2: LED_5V -> GND
- Rl31 pad 2: LED_5V -> GND
- Rl32 pad 2: LED_5V -> GND
- Rl4 pad 2: LED_5V -> GND
- Rl5 pad 2: LED_5V -> GND
- Rl6 pad 2: LED_5V -> GND
- Rl7 pad 2: LED_5V -> GND
- Rl8 pad 2: LED_5V -> GND
- Rl9 pad 2: LED_5V -> GND
- Rs1 pad 2: LED_5V -> GND
- Rs10 pad 2: LED_5V -> GND
- Rs11 pad 2: LED_5V -> GND
- Rs12 pad 2: LED_5V -> GND
- Rs13 pad 2: LED_5V -> GND
- Rs14 pad 2: LED_5V -> GND
- Rs15 pad 2: LED_5V -> GND
- Rs16 pad 2: LED_5V -> GND
- Rs17 pad 2: LED_5V -> GND
- Rs18 pad 2: LED_5V -> GND
- Rs19 pad 2: LED_5V -> GND
- Rs2 pad 2: LED_5V -> GND
- Rs20 pad 2: LED_5V -> GND
- Rs21 pad 2: LED_5V -> GND
- Rs22 pad 2: LED_5V -> GND
- Rs23 pad 2: LED_5V -> GND
- Rs24 pad 2: LED_5V -> GND
- Rs25 pad 2: LED_5V -> GND
- Rs26 pad 2: LED_5V -> GND
- Rs27 pad 2: LED_5V -> GND
- Rs28 pad 2: LED_5V -> GND
- Rs29 pad 2: LED_5V -> GND
- Rs3 pad 2: LED_5V -> GND
- Rs30 pad 2: LED_5V -> GND
- Rs31 pad 2: LED_5V -> GND
- Rs32 pad 2: LED_5V -> GND
- Rs4 pad 2: LED_5V -> GND
- Rs5 pad 2: LED_5V -> GND
- Rs6 pad 2: LED_5V -> GND
- Rs7 pad 2: LED_5V -> GND
- Rs8 pad 2: LED_5V -> GND
- Rs9 pad 2: LED_5V -> GND
- U1 pad 10: 1C -> Net-(Q3-E)
- U1 pad 12: LED_5V -> GND
- U1 pad 4: 1A -> Net-(Q1-E)
- U1 pad 6: 1B -> Net-(Q2-E)
- U1 pad 8: 1D -> Net-(Q4-E)
- U2 pad 10: 2C -> Net-(Q7-E)
- U2 pad 12: LED_5V -> GND
- U2 pad 4: 2A -> Net-(Q5-E)
- U2 pad 6: 2B -> Net-(Q6-E)
- U2 pad 8: 2D -> Net-(Q8-E)
- U3 pad 10: 3C -> Net-(Q11-E)
- U3 pad 12: LED_5V -> GND
- U3 pad 4: 3A -> Net-(Q9-E)
- U3 pad 6: 3B -> Net-(Q10-E)
- U3 pad 8: 3D -> Net-(Q12-E)
- U4 pad 10: 4C -> Net-(Q15-E)
- U4 pad 12: LED_5V -> GND
- U4 pad 4: 4A -> Net-(Q13-E)
- U4 pad 6: 4B -> Net-(Q14-E)
- U4 pad 8: 4D -> Net-(Q16-E)
- U5 pad 10: 5C -> Net-(Q25-E)
- U5 pad 12: LED_5V -> GND
- U5 pad 4: 5A -> Net-(Q17-E)
- U5 pad 6: 5B -> Net-(Q21-E)
- U5 pad 8: 5D -> Net-(Q29-E)
- U6 pad 10: 6C -> Net-(Q26-E)
- U6 pad 12: LED_5V -> GND
- U6 pad 4: 6A -> Net-(Q18-E)
- U6 pad 6: 6B -> Net-(Q22-E)
- U6 pad 8: 6D -> Net-(Q30-E)
- U7 pad 10: 7C -> Net-(Q27-E)
- U7 pad 12: LED_5V -> GND
- U7 pad 4: 7A -> Net-(Q19-E)
- U7 pad 6: 7B -> Net-(Q23-E)
- U7 pad 8: 7D -> Net-(Q31-E)
- U8 pad 10: 8C -> Net-(Q28-E)
- U8 pad 12: LED_5V -> GND
- U8 pad 4: 8A -> Net-(Q20-E)
- U8 pad 6: 8B -> Net-(Q24-E)
- U8 pad 8: 8D -> Net-(Q32-E)
Routing:
- net VCC: track 38.6 -> 1.26 mm
- net LED_5V: track 7.96 -> 1.17 mm, vias 3 -> 1
- net IMU_5V: track 0.00 -> 6.48 mm, vias 0 -> 1
- net 1: track 3.60 -> 0.00 mm
- net 4: track 3.48 -> 0.00 mm
- net GND: track 0.00 -> 3.26 mm, vias 0 -> 2
- net 2: track 2.88 -> 0.00 mm
- net 3: track 2.83 -> 0.00 mm
Other:
- board text added: "5v"
