File: KiCad/prot3/8.1バックアップ1/prot3.kicad_sch (KiCad schematic)
At the start: 198 parts, among them J1 Conn_01x02_Socket, J2 LED_SW, J3 Conn_01x04_Socket, Q1 Q_Photo_NPN, Q10 Q_Photo_NPN, Q11 Q_Photo_NPN, Q12 Q_Photo_NPN, Q13 Q_Photo_NPN, Q14 Q_Photo_NPN, Q15 Q_Photo_NPN, Q16 Q_Photo_NPN, Q17 Q_Photo_NPN, Q18 Q_Photo_NPN, Q19 Q_Photo_NPN, Q2 Q_Photo_NPN, Q20 Q_Photo_NPN, Q21 Q_Photo_NPN, Q22 Q_Photo_NPN, Q23 Q_Photo_NPN, Q24 Q_Photo_NPN, Q25 Q_Photo_NPN, Q26 Q_Photo_NPN, Q27 Q_Photo_NPN, Q28 Q_Photo_NPN, Q29 Q_Photo_NPN, Q3 Q_Photo_NPN, Q30 Q_Photo_NPN, Q31 Q_Photo_NPN, Q32 Q_Photo_NPN, Q4 Q_Photo_NPN, Q5 Q_Photo_NPN, Q6 Q_Photo_NPN, Q7 Q_Photo_NPN, Q8 Q_Photo_NPN, Q9 Q_Photo_NPN, U1 LM339, U2 LM339, U3 LM339, U4 LM339, U5 LM339, U6 LM339, U7 LM339, U8 LM339

Commit message: コンパレーターchに名札配置、rpzero仮完成
Connections:
- net 1A is gone; now on an unnamed net: U1.4 (-)
- net 1B is gone; now on an unnamed net: U1.6 (-)
- net 1C is gone; now on an unnamed net: U1.10 (-)
- net 1D is gone; now on an unnamed net: U1.8 (-)
- net 2A is gone; now on an unnamed net: U2.4 (-)
- net 2B is gone; now on an unnamed net: U2.6 (-)
- net 2C is gone; now on an unnamed net: U2.10 (-)
- net 2D is gone; now on an unnamed net: U2.8 (-)
- net 3A is gone; now on an unnamed net: U3.4 (-)
- net 3B is gone; now on an unnamed net: U3.6 (-)
- net 3C is gone; now on an unnamed net: U3.10 (-)
- net 3D is gone; now on an unnamed net: U3.8 (-)
- net 4A is gone; now on an unnamed net: U4.4 (-)
- net 4B is gone; now on an unnamed net: U4.6 (-)
- net 4C is gone; now on an unnamed net: U4.10 (-)
- net 4D is gone; now on an unnamed net: U4.8 (-)
- net 5A is gone; now on an unnamed net: U5.4 (-)
- net 5B is gone; now on an unnamed net: U5.6 (-)
- net 5C is gone; now on an unnamed net: U5.10 (-)
- net 5D is gone; now on an unnamed net: U5.8 (-)
- net 6A is gone; now on an unnamed net: U6.4 (-)
- net 6B is gone; now on an unnamed net: U6.6 (-)
- net 6C is gone; now on an unnamed net: U6.10 (-)
- net 6D is gone; now on an unnamed net: U6.8 (-)
- net 7A is gone; now on an unnamed net: U7.4 (-)
- net 7B is gone; now on an unnamed net: U7.6 (-)
- net 7C is gone; now on an unnamed net: U7.10 (-)
- net 7D is gone; now on an unnamed net: U7.8 (-)
- net 8A is gone; now on an unnamed net: U8.4 (-)
- net 8B is gone; now on an unnamed net: U8.6 (-)
- net 8C is gone; now on an unnamed net: U8.10 (-)
- net 8D is gone; now on an unnamed net: U8.8 (-)
- net GND: no longer C13.1, D1.2 (A), D10.2 (A), D11.2 (A), D12.2 (A), D13.2 (A), D14.2 (A), D15.2 (A), D16.2 (A), D17.2 (A), D18.2 (A), D19.2 (A), D2.2 (A), D20.2 (A), D21.2 (A), D22.2 (A), D23.2 (A), D24.2 (A), D25.2 (A), D26.2 (A), D27.2 (A), D28.2 (A), D29.2 (A), D3.2 (A), D30.2 (A), D31.2 (A), D32.2 (A), D4.2 (A), D5.2 (A), D6.2 (A), D7.2 (A), D8.2 (A), D9.2 (A), J1.1 (Pin_1), J2.3 (Pin_3)
- new net LED_5V: C13.1, D1.2 (A), D10.2 (A), D11.2 (A), D12.2 (A), D13.2 (A), D14.2 (A), D15.2 (A), D16.2 (A), D17.2 (A), D18.2 (A), D19.2 (A), D2.2 (A), D20.2 (A), D21.2 (A), D22.2 (A), D23.2 (A), D24.2 (A), D25.2 (A), D26.2 (A), D27.2 (A), D28.2 (A), D29.2 (A), D3.2 (A), D30.2 (A), D31.2 (A), D32.2 (A), D4.2 (A), D5.2 (A), D6.2 (A), D7.2 (A), D8.2 (A), D9.2 (A), J1.1 (Pin_1), J2.3 (Pin_3)
