File: KiCad/prot4/prot4.kicad_pcb (KiCad board)
At the start: 2 copper layers, 140 x 140 mm, 217 parts, among them J1 Conn_01x02_Socket, J2 LED_SW, J3 Conn_01x04_Socket, Q1 Q_Photo_NPN, Q10 Q_Photo_NPN, Q11 Q_Photo_NPN, Q12 Q_Photo_NPN, Q13 Q_Photo_NPN, Q14 Q_Photo_NPN, Q15 Q_Photo_NPN, Q16 Q_Photo_NPN, Q17 Q_Photo_NPN, Q18 Q_Photo_NPN, Q19 Q_Photo_NPN, Q2 Q_Photo_NPN, Q20 Q_Photo_NPN, Q21 Q_Photo_NPN, Q22 Q_Photo_NPN, Q23 Q_Photo_NPN, Q24 Q_Photo_NPN, Q25 Q_Photo_NPN, Q26 Q_Photo_NPN, Q27 Q_Photo_NPN, Q28 Q_Photo_NPN, Q29 Q_Photo_NPN, Q3 Q_Photo_NPN, Q30 Q_Photo_NPN, Q31 Q_Photo_NPN, Q32 Q_Photo_NPN, Q4 Q_Photo_NPN, Q5 Q_Photo_NPN, Q6 Q_Photo_NPN, Q7 Q_Photo_NPN, Q8 Q_Photo_NPN, Q9 Q_Photo_NPN, U1 LM393, U10 LM393, U11 LM393, U12 LM393, U13 LM393, U14 LM393, U15 LM393, U16 LM393, U2 LM393, U3 LM393, U4 LM393, U5 LM393, U6 LM393, U7 LM393, U8 LM393, U9 LM393

Commit message: 円形配置ほぼ完了
Parts:
- removed Rc10, Rc11, Rc12, Rc13, Rc14, Rc15, Rc16, Rc17, Rc18, Rc19, Rc20, Rc21, Rc22, Rc23, Rc24, Rc25, Rc26, Rc27, Rc28, Rc29, Rc3, Rc30, Rc31, Rc32, Rc4, Rc5, Rc6, Rc7, Rc8, Rc9, Rs10, Rs11, Rs12, Rs13, Rs14, Rs15, Rs16, Rs17, Rs18, Rs19, Rs20, Rs21, Rs22, Rs23, Rs24, Rs25, Rs26, Rs27, Rs28, Rs29, Rs3, Rs30, Rs31, Rs32, Rs4, Rs5, Rs6, Rs7, Rs8, Rs9: R, Resistor_SMD:R_0603_1608Metric_Pad0.98x0.95mm_HandSolder
- added Rca10: R, Resistor_SMD:R_0603_1608Metric_Pad0.98x0.95mm_HandSolder, F.Cu at (448.5, 523.9)
- added Rca11: R, Resistor_SMD:R_0603_1608Metric_Pad0.98x0.95mm_HandSolder, F.Cu at (461.6, 541.7)
- added Rca12: R, Resistor_SMD:R_0603_1608Metric_Pad0.98x0.95mm_HandSolder, F.Cu at (480.5, 553.3)
- added Rca13: R, Resistor_SMD:R_0603_1608Metric_Pad0.98x0.95mm_HandSolder, F.Cu at (502.4, 556.7)
- added Rca14: R, Resistor_SMD:R_0603_1608Metric_Pad0.98x0.95mm_HandSolder, F.Cu at (523.9, 551.5)
- added Rca15: R, Resistor_SMD:R_0603_1608Metric_Pad0.98x0.95mm_HandSolder, F.Cu at (541.7, 538.4)
- added Rca16: R, Resistor_SMD:R_0603_1608Metric_Pad0.98x0.95mm_HandSolder, F.Cu at (553.3, 519.5)
- added Rca2: R, Resistor_SMD:R_0603_1608Metric_Pad0.98x0.95mm_HandSolder, F.Cu at (551.5, 476.1)
- added Rca3: R, Resistor_SMD:R_0603_1608Metric_Pad0.98x0.95mm_HandSolder, F.Cu at (538.4, 458.3)
- added Rca4: R, Resistor_SMD:R_0603_1608Metric_Pad0.98x0.95mm_HandSolder, F.Cu at (519.5, 446.7)
- added Rca5: R, Resistor_SMD:R_0603_1608Metric_Pad0.98x0.95mm_HandSolder, F.Cu at (497.6, 443.3)
- added Rca6: R, Resistor_SMD:R_0603_1608Metric_Pad0.98x0.95mm_HandSolder, F.Cu at (476.1, 448.5)
- added Rca7: R, Resistor_SMD:R_0603_1608Metric_Pad0.98x0.95mm_HandSolder, F.Cu at (458.3, 461.6)
- added Rca8: R, Resistor_SMD:R_0603_1608Metric_Pad0.98x0.95mm_HandSolder, F.Cu at (446.7, 480.5)
- added Rca9: R, Resistor_SMD:R_0603_1608Metric_Pad0.98x0.95mm_HandSolder, F.Cu at (443.3, 502.4)
- added Rcb10: R, Resistor_SMD:R_0603_1608Metric_Pad0.98x0.95mm_HandSolder, F.Cu at (451.7, 532.4)
- added Rcb11: R, Resistor_SMD:R_0603_1608Metric_Pad0.98x0.95mm_HandSolder, F.Cu at (467.8, 548.4)
- added Rcb12: R, Resistor_SMD:R_0603_1608Metric_Pad0.98x0.95mm_HandSolder, F.Cu at (488.8, 557.0)
- added Rcb13: R, Resistor_SMD:R_0603_1608Metric_Pad0.98x0.95mm_HandSolder, F.Cu at (511.4, 557.0)
- added Rcb14: R, Resistor_SMD:R_0603_1608Metric_Pad0.98x0.95mm_HandSolder, F.Cu at (532.4, 548.3)
- added Rcb15: R, Resistor_SMD:R_0603_1608Metric_Pad0.98x0.95mm_HandSolder, F.Cu at (548.4, 532.2)
- added Rcb16: R, Resistor_SMD:R_0603_1608Metric_Pad0.98x0.95mm_HandSolder, F.Cu at (557.0, 511.2)
- added Rcb2: R, Resistor_SMD:R_0603_1608Metric_Pad0.98x0.95mm_HandSolder, F.Cu at (548.3, 467.6)
- added Rcb3: R, Resistor_SMD:R_0603_1608Metric_Pad0.98x0.95mm_HandSolder, F.Cu at (532.2, 451.6)
- added Rcb4: R, Resistor_SMD:R_0603_1608Metric_Pad0.98x0.95mm_HandSolder, F.Cu at (511.2, 443.0)
- added Rcb5: R, Resistor_SMD:R_0603_1608Metric_Pad0.98x0.95mm_HandSolder, F.Cu at (488.6, 443.0)
- added Rcb6: R, Resistor_SMD:R_0603_1608Metric_Pad0.98x0.95mm_HandSolder, F.Cu at (467.6, 451.7)
- added Rcb7: R, Resistor_SMD:R_0603_1608Metric_Pad0.98x0.95mm_HandSolder, F.Cu at (451.6, 467.8)
- added Rcb8: R, Resistor_SMD:R_0603_1608Metric_Pad0.98x0.95mm_HandSolder, F.Cu at (443.0, 488.8)
- added Rcb9: R, Resistor_SMD:R_0603_1608Metric_Pad0.98x0.95mm_HandSolder, F.Cu at (443.0, 511.4)
- added Rsa10: R, Resistor_SMD:R_0603_1608Metric_Pad0.98x0.95mm_HandSolder, F.Cu at (439.3, 530.6)
- added Rsa11: R, Resistor_SMD:R_0603_1608Metric_Pad0.98x0.95mm_HandSolder, F.Cu at (455.6, 551.5)
- added Rsa12: R, Resistor_SMD:R_0603_1608Metric_Pad0.98x0.95mm_HandSolder, F.Cu at (478.6, 564.6)
- added Rsa13: R, Resistor_SMD:R_0603_1608Metric_Pad0.98x0.95mm_HandSolder, F.Cu at (505.0, 567.8)
- added Rsa14: R, Resistor_SMD:R_0603_1608Metric_Pad0.98x0.95mm_HandSolder, F.Cu at (530.6, 560.7)
- added Rsa15: R, Resistor_SMD:R_0603_1608Metric_Pad0.98x0.95mm_HandSolder, F.Cu at (551.5, 544.4)
- added Rsa16: R, Resistor_SMD:R_0603_1608Metric_Pad0.98x0.95mm_HandSolder, F.Cu at (564.6, 521.4)
- added Rsa2: R, Resistor_SMD:R_0603_1608Metric_Pad0.98x0.95mm_HandSolder, F.Cu at (560.7, 469.4)
- added Rsa3: R, Resistor_SMD:R_0603_1608Metric_Pad0.98x0.95mm_HandSolder, F.Cu at (544.4, 448.5)
- added Rsa4: R, Resistor_SMD:R_0603_1608Metric_Pad0.98x0.95mm_HandSolder, F.Cu at (521.4, 435.4)
- added Rsa5: R, Resistor_SMD:R_0603_1608Metric_Pad0.98x0.95mm_HandSolder, F.Cu at (495.0, 432.2)
- added Rsa6: R, Resistor_SMD:R_0603_1608Metric_Pad0.98x0.95mm_HandSolder, F.Cu at (469.4, 439.3)
- added Rsa7: R, Resistor_SMD:R_0603_1608Metric_Pad0.98x0.95mm_HandSolder, F.Cu at (448.5, 455.6)
- added Rsa8: R, Resistor_SMD:R_0603_1608Metric_Pad0.98x0.95mm_HandSolder, F.Cu at (435.4, 478.6)
- added Rsa9: R, Resistor_SMD:R_0603_1608Metric_Pad0.98x0.95mm_HandSolder, F.Cu at (432.2, 505.0)
- added Rsb10: R, Resistor_SMD:R_0603_1608Metric_Pad0.98x0.95mm_HandSolder, F.Cu at (447.4, 543.1)
- added Rsb11: R, Resistor_SMD:R_0603_1608Metric_Pad0.98x0.95mm_HandSolder, F.Cu at (467.9, 560.0)
- added Rsb12: R, Resistor_SMD:R_0603_1608Metric_Pad0.98x0.95mm_HandSolder, F.Cu at (493.3, 567.7)
- added Rsb13: R, Resistor_SMD:R_0603_1608Metric_Pad0.98x0.95mm_HandSolder, F.Cu at (519.7, 565.1)
- added Rsb14: R, Resistor_SMD:R_0603_1608Metric_Pad0.98x0.95mm_HandSolder, F.Cu at (543.1, 552.6)
- added Rsb15: R, Resistor_SMD:R_0603_1608Metric_Pad0.98x0.95mm_HandSolder, F.Cu at (560.0, 532.1)
- added Rsb16: R, Resistor_SMD:R_0603_1608Metric_Pad0.98x0.95mm_HandSolder, F.Cu at (567.7, 506.7)
- added Rsb2: R, Resistor_SMD:R_0603_1608Metric_Pad0.98x0.95mm_HandSolder, F.Cu at (552.6, 456.9)
- added Rsb3: R, Resistor_SMD:R_0603_1608Metric_Pad0.98x0.95mm_HandSolder, F.Cu at (532.1, 440.0)
- added Rsb4: R, Resistor_SMD:R_0603_1608Metric_Pad0.98x0.95mm_HandSolder, F.Cu at (506.7, 432.3)
- added Rsb5: R, Resistor_SMD:R_0603_1608Metric_Pad0.98x0.95mm_HandSolder, F.Cu at (480.3, 434.9)
- added Rsb6: R, Resistor_SMD:R_0603_1608Metric_Pad0.98x0.95mm_HandSolder, F.Cu at (456.9, 447.4)
- added Rsb7: R, Resistor_SMD:R_0603_1608Metric_Pad0.98x0.95mm_HandSolder, F.Cu at (440.0, 467.9)
- added Rsb8: R, Resistor_SMD:R_0603_1608Metric_Pad0.98x0.95mm_HandSolder, F.Cu at (432.3, 493.3)
- added Rsb9: R, Resistor_SMD:R_0603_1608Metric_Pad0.98x0.95mm_HandSolder, F.Cu at (434.9, 519.7)
- moved Q5 229.2 mm to (548.1, 451.9), turned to -45 degrees
- moved Q4 228.4 mm to (556.5, 462.2), turned to -56.25 degrees
- moved Q6 228.4 mm to (537.8, 443.5), turned to -33.75 degrees
- moved U2 227.3 mm to (554.1, 471.2), turned to 123.52 degrees
- moved Q3 226.0 mm to (562.8, 474.0), turned to -67.5 degrees
- moved Q7 226.0 mm to (526.0, 437.2), turned to -22.5 degrees
- moved U3 224.7 mm to (538.9, 452.7), turned to 146.02 degrees
- moved Q8 222.1 mm to (513.3, 433.3), turned to -11.25 degrees
- moved U4 216.9 mm to (517.9, 441.4), turned to 168.52 degrees
- moved Q9 216.7 mm to (500.0, 432.0)
- moved Q10 209.9 mm to (486.7, 433.3), turned to 11.25 degrees
- moved C16 205.5 mm to (554.2, 515.0), turned to -99.978 degrees
- moved Q32 205.5 mm to (566.7, 513.3), turned to -101.25 degrees
- moved U16 204.4 mm to (558.6, 517.9), turned to 78.52 degrees
- moved U5 204.3 mm to (494.1, 439.1), turned to -168.98 degrees
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- renumbered Rc1 to Rca1, Rc2 to Rcb1, Rs1 to Rsa1, Rs2 to Rsb1
Routing:
- net GND: track 48.6 -> 30043.2 mm, vias 2 -> 4337
- net VCC: track 43.1 -> 673.6 mm
- net Net-(Q1-E): track 21.1 -> 251.0 mm
- net Net-(Q2-E): track 19.5 -> 172.3 mm
- net conp_+: track 6.21 -> 63.9 mm, vias 2 -> 32
- net LED_5V: track 9.55 -> 65.1 mm, vias 2 -> 17
- net Net-(D30-K): track 0.00 -> 50.3 mm
- net Net-(D22-K): track 0.00 -> 50.3 mm
- net Net-(D6-K): track 0.00 -> 50.3 mm
- net Net-(D14-K): track 0.00 -> 50.3 mm
- net Net-(D10-K): track 0.00 -> 50.3 mm
- net Net-(D18-K): track 0.00 -> 50.3 mm
- net Net-(D26-K): track 0.00 -> 50.3 mm
- net Net-(D12-K): track 0.00 -> 50.3 mm
- net Net-(D4-K): track 0.00 -> 50.3 mm
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