File: KiCad/prot4/prot4.kicad_sch (KiCad schematic)
At the start: 217 parts, among them J1 Conn_01x02_Socket, J2 LED_SW, J3 Conn_01x04_Socket, Q1 Q_Photo_NPN, Q10 Q_Photo_NPN, Q11 Q_Photo_NPN, Q12 Q_Photo_NPN, Q13 Q_Photo_NPN, Q14 Q_Photo_NPN, Q15 Q_Photo_NPN, Q16 Q_Photo_NPN, Q17 Q_Photo_NPN, Q18 Q_Photo_NPN, Q19 Q_Photo_NPN, Q2 Q_Photo_NPN, Q20 Q_Photo_NPN, Q21 Q_Photo_NPN, Q22 Q_Photo_NPN, Q23 Q_Photo_NPN, Q24 Q_Photo_NPN, Q25 Q_Photo_NPN, Q26 Q_Photo_NPN, Q27 Q_Photo_NPN, Q28 Q_Photo_NPN, Q29 Q_Photo_NPN, Q3 Q_Photo_NPN, Q30 Q_Photo_NPN, Q31 Q_Photo_NPN, Q32 Q_Photo_NPN, Q4 Q_Photo_NPN, Q5 Q_Photo_NPN, Q6 Q_Photo_NPN, Q7 Q_Photo_NPN, Q8 Q_Photo_NPN, Q9 Q_Photo_NPN, U1 LM393, U10 LM393, U11 LM393, U12 LM393, U13 LM393, U14 LM393, U15 LM393, U16 LM393, U2 LM393, U3 LM393, U4 LM393, U5 LM393, U6 LM393, U7 LM393, U8 LM393, U9 LM393

Commit message: 円形配置ほぼ完了
Parts:
- removed Rc10, Rc11, Rc12, Rc13, Rc14, Rc15, Rc16, Rc17, Rc18, Rc19, Rc20, Rc21, Rc22, Rc23, Rc24, Rc25, Rc26, Rc27, Rc28, Rc29, Rc3, Rc30, Rc31, Rc32, Rc4, Rc5, Rc6, Rc7, Rc8, Rc9, Rs10, Rs11, Rs12, Rs13, Rs14, Rs15, Rs16, Rs17, Rs18, Rs19, Rs20, Rs21, Rs22, Rs23, Rs24, Rs25, Rs26, Rs27, Rs28, Rs29, Rs3, Rs30, Rs31, Rs32, Rs4, Rs5, Rs6, Rs7, Rs8, Rs9: R, Resistor_SMD:R_0603_1608Metric_Pad0.98x0.95mm_HandSolder, symbol Device:R
- added Rca10, Rca11, Rca12, Rca13, Rca14, Rca15, Rca16, Rca2, Rca3, Rca4, Rca5, Rca6, Rca7, Rca8, Rca9, Rcb10, Rcb11, Rcb12, Rcb13, Rcb14, Rcb15, Rcb16, Rcb2, Rcb3, Rcb4, Rcb5, Rcb6, Rcb7, Rcb8, Rcb9, Rsa10, Rsa11, Rsa12, Rsa13, Rsa14, Rsa15, Rsa16, Rsa2, Rsa3, Rsa4, Rsa5, Rsa6, Rsa7, Rsa8, Rsa9, Rsb10, Rsb11, Rsb12, Rsb13, Rsb14, Rsb15, Rsb16, Rsb2, Rsb3, Rsb4, Rsb5, Rsb6, Rsb7, Rsb8, Rsb9: R, Resistor_SMD:R_0603_1608Metric_Pad0.98x0.95mm_HandSolder, symbol Device:R
- renumbered C9 to C17, C11 to C18, C12 to C19, C10 to C20, C16 to C21, C17 to C22, C13 to C23, C18 to C24, C14 to C25, C15 to C26, Rc1 to Rca1, Rc2 to Rcb1, Rs1 to Rsa1, Rs2 to Rsb1
Connections:
- net 1: now also Rca10.1, Rca11.1, Rca12.1, Rca13.1, Rca14.1, Rca15.1, Rca16.1, Rca2.1, Rca3.1, Rca4.1, Rca5.1, Rca6.1, Rca7.1, Rca8.1, Rca9.1
- net 2: now also Rcb10.1, Rcb11.1, Rcb12.1, Rcb13.1, Rcb14.1, Rcb15.1, Rcb16.1, Rcb2.1, Rcb3.1, Rcb4.1, Rcb5.1, Rcb6.1, Rcb7.1, Rcb8.1, Rcb9.1
- net GND: now also Rsa10.1, Rsa11.1, Rsa12.1, Rsa13.1, Rsa14.1, Rsa15.1, Rsa16.1, Rsa2.1, Rsa3.1, Rsa4.1, Rsa5.1, Rsa6.1, Rsa7.1, Rsa8.1, Rsa9.1, Rsb10.1, Rsb11.1, Rsb12.1, Rsb13.1, Rsb14.1, Rsb15.1, Rsb16.1, Rsb2.1, Rsb3.1, Rsb4.1, Rsb5.1, Rsb6.1, Rsb7.1, Rsb8.1, Rsb9.1
- net VCC: now also Rca10.2, Rca11.2, Rca12.2, Rca13.2, Rca14.2, Rca15.2, Rca16.2, Rca2.2, Rca3.2, Rca4.2, Rca5.2, Rca6.2, Rca7.2, Rca8.2, Rca9.2, Rcb10.2, Rcb11.2, Rcb12.2, Rcb13.2, Rcb14.2, Rcb15.2, Rcb16.2, Rcb2.2, Rcb3.2, Rcb4.2, Rcb5.2, Rcb6.2, Rcb7.2, Rcb8.2, Rcb9.2
- net at Q23.2 (E), U11.6 (-): now also Rsb11.2
- net at Q22.2 (E), U10.6 (-): now also Rsb10.2
- net at Q11.2 (E), U7.2 (-): now also Rsa7.2
- net at Q9.2 (E), U5.2 (-): now also Rsa5.2
- net at Q20.2 (E), U12.2 (-): now also Rsa12.2
- net at Q5.2 (E), U3.2 (-): now also Rsa3.2
- net at Q17.2 (E), U9.2 (-): now also Rsa9.2
- net at Q13.2 (E), U5.6 (-): now also Rsb5.2
- net at Q6.2 (E), U3.6 (-): now also Rsb3.2
- net at Q26.2 (E), U14.2 (-): now also Rsa14.2
- net at Q29.2 (E), U13.6 (-): now also Rsb13.2
- net at Q8.2 (E), U4.6 (-): now also Rsb4.2
- net at Q25.2 (E), U13.2 (-): now also Rsa13.2
- net at Q21.2 (E), U9.6 (-): now also Rsb9.2
- net at Q31.2 (E), U15.6 (-): now also Rsb15.2
- net at Q7.2 (E), U4.2 (-): now also Rsa4.2
- net at Q15.2 (E), U7.6 (-): now also Rsb7.2
- net at Q14.2 (E), U6.6 (-): now also Rsb6.2
- net at Q27.2 (E), U15.2 (-): now also Rsa15.2
- net at Q19.2 (E), U11.2 (-): now also Rsa11.2
- net at Q18.2 (E), U10.2 (-): now also Rsa10.2
- net at Q3.2 (E), U2.2 (-): now also Rsa2.2
- net at Q16.2 (E), U8.6 (-): now also Rsb8.2
- net at Q24.2 (E), U12.6 (-): now also Rsb12.2
- net at Q4.2 (E), U2.6 (-): now also Rsb2.2
- net at Q32.2 (E), U16.6 (-): now also Rsb16.2
- net at Q12.2 (E), U8.2 (-): now also Rsa8.2
- net at Q28.2 (E), U16.2 (-): now also Rsa16.2
- net at Q30.2 (E), U14.6 (-): now also Rsb14.2
- net at Q10.2 (E), U6.2 (-): now also Rsa6.2
