File: KiCad/prot4/_autosave-prot4.kicad_pcb (KiCad board)
At the start: 2 copper layers, 140 x 140 mm, 217 parts, among them J1 Conn_01x02_Socket, J2 LED_SW, J3 Conn_01x04_Socket, Q1 Q_Photo_NPN, Q10 Q_Photo_NPN, Q11 Q_Photo_NPN, Q12 Q_Photo_NPN, Q13 Q_Photo_NPN, Q14 Q_Photo_NPN, Q15 Q_Photo_NPN, Q16 Q_Photo_NPN, Q17 Q_Photo_NPN, Q18 Q_Photo_NPN, Q19 Q_Photo_NPN, Q2 Q_Photo_NPN, Q20 Q_Photo_NPN, Q21 Q_Photo_NPN, Q22 Q_Photo_NPN, Q23 Q_Photo_NPN, Q24 Q_Photo_NPN, Q25 Q_Photo_NPN, Q26 Q_Photo_NPN, Q27 Q_Photo_NPN, Q28 Q_Photo_NPN, Q29 Q_Photo_NPN, Q3 Q_Photo_NPN, Q30 Q_Photo_NPN, Q31 Q_Photo_NPN, Q32 Q_Photo_NPN, Q4 Q_Photo_NPN, Q5 Q_Photo_NPN, Q6 Q_Photo_NPN, Q7 Q_Photo_NPN, Q8 Q_Photo_NPN, Q9 Q_Photo_NPN, U1 LM393, U10 LM393, U11 LM393, U12 LM393, U13 LM393, U14 LM393, U15 LM393, U16 LM393, U2 LM393, U3 LM393, U4 LM393, U5 LM393, U6 LM393, U7 LM393, U8 LM393, U9 LM393

Commit message: 重すぎ
Parts:
- moved RP2040_Zero1 200.8 mm to (530.0, 479.0), turned to 90 degrees
- moved J3 167.9 mm to (503.0, 493.0), turned to 180 degrees
- moved RP2040_Zero2 32.1 mm to (530.0, 521.0)
