File: KiCad/prot4/ネット減らしたい/prot4/prot4.kicad_sch (KiCad schematic)
At the start: 217 parts, among them J1 Conn_01x02_Socket, J2 LED_SW, J3 Conn_01x04_Socket, Q1 Q_Photo_NPN, Q10 Q_Photo_NPN, Q11 Q_Photo_NPN, Q12 Q_Photo_NPN, Q13 Q_Photo_NPN, Q14 Q_Photo_NPN, Q15 Q_Photo_NPN, Q16 Q_Photo_NPN, Q17 Q_Photo_NPN, Q18 Q_Photo_NPN, Q19 Q_Photo_NPN, Q2 Q_Photo_NPN, Q20 Q_Photo_NPN, Q21 Q_Photo_NPN, Q22 Q_Photo_NPN, Q23 Q_Photo_NPN, Q24 Q_Photo_NPN, Q25 Q_Photo_NPN, Q26 Q_Photo_NPN, Q27 Q_Photo_NPN, Q28 Q_Photo_NPN, Q29 Q_Photo_NPN, Q3 Q_Photo_NPN, Q30 Q_Photo_NPN, Q31 Q_Photo_NPN, Q32 Q_Photo_NPN, Q4 Q_Photo_NPN, Q5 Q_Photo_NPN, Q6 Q_Photo_NPN, Q7 Q_Photo_NPN, Q8 Q_Photo_NPN, Q9 Q_Photo_NPN, U1 LM393, U10 LM393, U11 LM393, U12 LM393, U13 LM393, U14 LM393, U15 LM393, U16 LM393, U2 LM393, U3 LM393, U4 LM393, U5 LM393, U6 LM393, U7 LM393, U8 LM393, U9 LM393

Commit message: 部品に配線開始
Connections:
- net 1: no longer RP2040_Zero1.20 (29), Rca10.1, Rca11.1, Rca12.1, Rca13.1, Rca14.1, Rca15.1, Rca16.1, Rca2.1, Rca3.1, Rca4.1, Rca5.1, Rca6.1, Rca7.1, Rca8.1, Rca9.1, U10.1, U11.1, U12.1, U13.1, U14.1, U15.1, U16.1, U2.1, U3.1, U4.1, U5.1, U6.1, U7.1, U8.1, U9.1
- net 10: now also Rcb5.1, U5.7
- net 11: now also Rca6.1, U6.1
- net 12: now also Rcb6.1, U6.7
- net 13: now also Rca7.1, U7.1
- net 14: now also Rcb7.1, U7.7
- net 15: now also Rca8.1, U8.1
- net 16: now also Rcb8.1, U8.7
- net 17: now also Rca9.1, U9.1
- net 18: now also Rcb9.1, U9.7
- net 19: now also Rca10.1, U10.1
- net 2: no longer RP2040_Zero1.19 (28), Rcb10.1, Rcb11.1, Rcb12.1, Rcb13.1, Rcb14.1, Rcb15.1, Rcb16.1, Rcb2.1, Rcb3.1, Rcb4.1, Rcb5.1, Rcb6.1, Rcb7.1, Rcb8.1, Rcb9.1, U10.7, U11.7, U12.7, U13.7, U14.7, U15.7, U16.7, U2.7, U3.7, U4.7, U5.7, U6.7, U7.7, U8.7, U9.7
- net 20: now also Rcb10.1, U10.7
- net 21: now also Rca11.1, U11.1
- net 22: now also Rcb11.1, U11.7
- net 23: now also Rca12.1, U12.1
- net 24: now also Rcb12.1, U12.7
- net 25: now also Rca13.1, U13.1
- net 26: now also Rcb13.1, U13.7
- net 27: now also Rca14.1, U14.1
- net 28: now also Rcb14.1, U14.7
- net 29: now also Rca15.1, U15.1
- net 3: now also Rca2.1, U2.1; no longer RP2040_Zero1.17 (26)
- net 30: now also Rcb15.1, U15.7
- net 31: now also Rca16.1, U16.1
- net 32: now also Rcb16.1, U16.7
- net 4: now also Rcb2.1, U2.7; no longer RP2040_Zero1.18 (27)
- net 5: now also Rca3.1, U3.1; no longer RP2040_Zero1.16 (15)
- net 6: now also Rcb3.1, U3.7; no longer RP2040_Zero1.15 (14)
- net 7: now also Rca4.1, U4.1; no longer RP2040_Zero1.10 (9)
- net 8: now also Rcb4.1, U4.7; no longer RP2040_Zero1.11 (10)
- net 9: now also Rca5.1, U5.1
- net LED_5V: no longer C21.1, C22.1
- net VCC: now also Rca14.2, Rcb14.2
- net at Rsb14.2, U14.6 (-): now also Q28.2 (E); no longer Q30.2 (E)
- net at Rsb13.2, U13.6 (-): now also Q26.2 (E); no longer Q29.2 (E)
- net at Rsa7.2, U7.2 (-): now also Q13.2 (E); no longer Q11.2 (E)
- net at Rsa12.2, U12.2 (-): now also Q23.2 (E); no longer Q20.2 (E)
- net at Rsa8.2, U8.2 (-): now also Q15.2 (E); no longer Q12.2 (E)
- net at Rsb9.2, U9.6 (-): now also Q18.2 (E); no longer Q21.2 (E)
- net at Rsb11.2, U11.6 (-): now also Q22.2 (E); no longer Q23.2 (E)
- net at Rsa16.2, U16.2 (-): now also Q31.2 (E); no longer Q28.2 (E)
- net at Rsb6.2, U6.6 (-): now also Q12.2 (E); no longer Q14.2 (E)
- net at J1.1 (Pin_1), J2.2 (Pin_2), J2.3 (Pin_3): now also C21.1, C22.1
- net at Rsa14.2, U14.2 (-): now also Q27.2 (E); no longer Q26.2 (E)
- net at Rsb10.2, U10.6 (-): now also Q20.2 (E); no longer Q22.2 (E)
- net at Rsa15.2, U15.2 (-): now also Q29.2 (E); no longer Q27.2 (E)
- net at Rsb5.2, U5.6 (-): now also Q10.2 (E); no longer Q13.2 (E)
- net at Rsa11.2, U11.2 (-): now also Q21.2 (E); no longer Q19.2 (E)
- net at Rsb15.2, U15.6 (-): now also Q30.2 (E); no longer Q31.2 (E)
- net at Rsa6.2, U6.2 (-): now also Q11.2 (E); no longer Q10.2 (E)
- net at Rsb7.2, U7.6 (-): now also Q14.2 (E); no longer Q15.2 (E)
- net at Rsa10.2, U10.2 (-): now also Q19.2 (E); no longer Q18.2 (E)
Other:
- moved on the sheet: C21, C22, Q10, Q11, Q12, Q13, Q14, Q15, Q18, Q19, Q20, Q21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
