File: KiCad/prot4/ネット減らしたい/prot4/prot4.kicad_pcb (KiCad board)
At the start: 2 copper layers, 140 x 140 mm, 217 parts, among them J1 Conn_01x02_Socket, J2 LED_SW, J3 Conn_01x04_Socket, Q1 Q_Photo_NPN, Q10 Q_Photo_NPN, Q11 Q_Photo_NPN, Q12 Q_Photo_NPN, Q13 Q_Photo_NPN, Q14 Q_Photo_NPN, Q15 Q_Photo_NPN, Q16 Q_Photo_NPN, Q17 Q_Photo_NPN, Q18 Q_Photo_NPN, Q19 Q_Photo_NPN, Q2 Q_Photo_NPN, Q20 Q_Photo_NPN, Q21 Q_Photo_NPN, Q22 Q_Photo_NPN, Q23 Q_Photo_NPN, Q24 Q_Photo_NPN, Q25 Q_Photo_NPN, Q26 Q_Photo_NPN, Q27 Q_Photo_NPN, Q28 Q_Photo_NPN, Q29 Q_Photo_NPN, Q3 Q_Photo_NPN, Q30 Q_Photo_NPN, Q31 Q_Photo_NPN, Q32 Q_Photo_NPN, Q4 Q_Photo_NPN, Q5 Q_Photo_NPN, Q6 Q_Photo_NPN, Q7 Q_Photo_NPN, Q8 Q_Photo_NPN, Q9 Q_Photo_NPN, U1 LM393, U10 LM393, U11 LM393, U12 LM393, U13 LM393, U14 LM393, U15 LM393, U16 LM393, U2 LM393, U3 LM393, U4 LM393, U5 LM393, U6 LM393, U7 LM393, U8 LM393, U9 LM393

Commit message: 部品に配線開始
Parts:
- J1, J3: moved to B.Cu
- moved B1 237.9 mm to (532.5, 499.8)
- moved C23 232.7 mm to (531.7, 507.1)
- moved C19 232.1 mm to (529.4, 476.5)
- moved C20 232.1 mm to (529.7, 481.1)
- moved C24 229.9 mm to (528.5, 502.2)
- moved RP2040_Zero1 226.5 mm to (530.0, 521.0), turned to 90 degrees
- moved C26 225.9 mm to (529.3, 483.0)
- moved R1 224.0 mm to (527.4, 497.4)
- moved C17 213.7 mm to (512.8, 505.1)
- moved C18 213.7 mm to (512.8, 507.6)
- moved C25 213.7 mm to (512.8, 525.2)
- moved RP2040_Zero2 211.0 mm to (530.0, 479.0), turned to 90 degrees
- moved LS1 208.1 mm to (542.1, 500.5)
- moved C21 203.3 mm to (494.8, 565.2)
- moved C22 201.9 mm to (494.8, 562.3)
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Connections:
- C21 pad 1: LED_5V -> Net-(J1-Pin_1)
- C22 pad 1: LED_5V -> Net-(J1-Pin_1)
- RP2040_Zero1 pad 10: 7 -> unconnected-(RP2040_Zero1-9-Pad10)
- RP2040_Zero1 pad 11: 8 -> unconnected-(RP2040_Zero1-10-Pad11)
- RP2040_Zero1 pad 15: 6 -> unconnected-(RP2040_Zero1-14-Pad15)
- RP2040_Zero1 pad 16: 5 -> unconnected-(RP2040_Zero1-15-Pad16)
- RP2040_Zero1 pad 17: 3 -> unconnected-(RP2040_Zero1-26-Pad17)
- RP2040_Zero1 pad 18: 4 -> unconnected-(RP2040_Zero1-27-Pad18)
- RP2040_Zero1 pad 19: 2 -> unconnected-(RP2040_Zero1-28-Pad19)
- RP2040_Zero1 pad 20: 1 -> unconnected-(RP2040_Zero1-29-Pad20)
- Rca10 pad 1: 1 -> 19
- Rca11 pad 1: 1 -> 21
- Rca12 pad 1: 1 -> 23
- Rca13 pad 1: 1 -> 25
- Rca14 pad 1: 1 -> 27
- Rca14 pad 2: unconnected-(Rca14-Pad2) -> VCC
- Rca15 pad 1: 1 -> 29
- Rca16 pad 1: 1 -> 31
- Rca2 pad 1: 1 -> 3
- Rca3 pad 1: 1 -> 5
- Rca4 pad 1: 1 -> 7
- Rca5 pad 1: 1 -> 9
- Rca6 pad 1: 1 -> 11
- Rca7 pad 1: 1 -> 13
- Rca8 pad 1: 1 -> 15
- Rca9 pad 1: 1 -> 17
- Rcb10 pad 1: 2 -> 20
- Rcb11 pad 1: 2 -> 22
- Rcb12 pad 1: 2 -> 24
- Rcb13 pad 1: 2 -> 26
- Rcb14 pad 1: 2 -> 28
- Rcb14 pad 2: unconnected-(Rcb14-Pad2) -> VCC
- Rcb15 pad 1: 2 -> 30
- Rcb16 pad 1: 2 -> 32
- Rcb2 pad 1: 2 -> 4
- Rcb3 pad 1: 2 -> 6
- Rcb4 pad 1: 2 -> 8
- Rcb5 pad 1: 2 -> 10
- Rcb6 pad 1: 2 -> 12
- Rcb7 pad 1: 2 -> 14
- Rcb8 pad 1: 2 -> 16
- Rcb9 pad 1: 2 -> 18
- Rsa10 pad 2: Net-(Q18-E) -> Net-(Q19-E)
- Rsa11 pad 2: Net-(Q19-E) -> Net-(Q21-E)
- Rsa12 pad 2: Net-(Q20-E) -> Net-(Q23-E)
- Rsa14 pad 2: Net-(Q26-E) -> Net-(Q27-E)
- Rsa15 pad 2: Net-(Q27-E) -> Net-(Q29-E)
- Rsa16 pad 2: Net-(Q28-E) -> Net-(Q31-E)
- Rsa6 pad 2: Net-(Q10-E) -> Net-(Q11-E)
- Rsa7 pad 2: Net-(Q11-E) -> Net-(Q13-E)
- Rsa8 pad 2: Net-(Q12-E) -> Net-(Q15-E)
- Rsb10 pad 2: Net-(Q22-E) -> Net-(Q20-E)
- Rsb11 pad 2: Net-(Q23-E) -> Net-(Q22-E)
- Rsb13 pad 2: Net-(Q29-E) -> Net-(Q26-E)
- Rsb14 pad 2: Net-(Q30-E) -> Net-(Q28-E)
- Rsb15 pad 2: Net-(Q31-E) -> Net-(Q30-E)
- Rsb5 pad 2: Net-(Q13-E) -> Net-(Q10-E)
- Rsb6 pad 2: Net-(Q14-E) -> Net-(Q12-E)
- Rsb7 pad 2: Net-(Q15-E) -> Net-(Q14-E)
- Rsb9 pad 2: Net-(Q21-E) -> Net-(Q18-E)
- U10 pad 1: 1 -> 19
- U10 pad 2: Net-(Q18-E) -> Net-(Q19-E)
- U10 pad 6: Net-(Q22-E) -> Net-(Q20-E)
- U10 pad 7: 2 -> 20
- U11 pad 1: 1 -> 21
- U11 pad 2: Net-(Q19-E) -> Net-(Q21-E)
- U11 pad 6: Net-(Q23-E) -> Net-(Q22-E)
- U11 pad 7: 2 -> 22
- U12 pad 1: 1 -> 23
- U12 pad 2: Net-(Q20-E) -> Net-(Q23-E)
- U12 pad 7: 2 -> 24
- U13 pad 1: 1 -> 25
- U13 pad 6: Net-(Q29-E) -> Net-(Q26-E)
- U13 pad 7: 2 -> 26
- U14 pad 1: 1 -> 27
- U14 pad 2: Net-(Q26-E) -> Net-(Q27-E)
- U14 pad 6: Net-(Q30-E) -> Net-(Q28-E)
- U14 pad 7: 2 -> 28
- U15 pad 1: 1 -> 29
- U15 pad 2: Net-(Q27-E) -> Net-(Q29-E)
- U15 pad 6: Net-(Q31-E) -> Net-(Q30-E)
- U15 pad 7: 2 -> 30
- U16 pad 1: 1 -> 31
- U16 pad 2: Net-(Q28-E) -> Net-(Q31-E)
- U16 pad 7: 2 -> 32
- U2 pad 1: 1 -> 3
- U2 pad 7: 2 -> 4
- U3 pad 1: 1 -> 5
- U3 pad 7: 2 -> 6
- U4 pad 1: 1 -> 7
- U4 pad 7: 2 -> 8
- U5 pad 1: 1 -> 9
- U5 pad 6: Net-(Q13-E) -> Net-(Q10-E)
- U5 pad 7: 2 -> 10
- U6 pad 1: 1 -> 11
- U6 pad 2: Net-(Q10-E) -> Net-(Q11-E)
- U6 pad 6: Net-(Q14-E) -> Net-(Q12-E)
- U6 pad 7: 2 -> 12
- U7 pad 1: 1 -> 13
- U7 pad 2: Net-(Q11-E) -> Net-(Q13-E)
- U7 pad 6: Net-(Q15-E) -> Net-(Q14-E)
- U7 pad 7: 2 -> 14
- U8 pad 1: 1 -> 15
- U8 pad 2: Net-(Q12-E) -> Net-(Q15-E)
- U8 pad 7: 2 -> 16
- U9 pad 1: 1 -> 17
- U9 pad 6: Net-(Q21-E) -> Net-(Q18-E)
- U9 pad 7: 2 -> 18
Routing:
- net GND: track 48.5 -> 829.3 mm, vias 2 -> 64
- net VCC: track 43.1 -> 729.1 mm
- net LED_5V: track 9.55 -> 202.0 mm, vias 2 -> 32
- net conp_+: track 6.21 -> 95.2 mm, vias 2 -> 32
- net Net-(J1-Pin_1): track 0.00 -> 29.6 mm, vias 0 -> 1
- net 6: track 0.00 -> 25.4 mm, vias 0 -> 1
- net Net-(Q29-E): track 0.00 -> 21.8 mm
- net Net-(Q21-E): track 0.00 -> 21.8 mm
- net Net-(Q5-E): track 0.00 -> 21.8 mm
- net Net-(Q13-E): track 0.00 -> 21.8 mm
- net Net-(Q31-E): track 0.00 -> 21.8 mm
- net Net-(Q7-E): track 0.00 -> 21.8 mm
- net Net-(Q23-E): track 0.00 -> 21.8 mm
- net Net-(Q15-E): track 0.00 -> 21.8 mm
- net Net-(Q25-E): track 0.00 -> 21.8 mm
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
Commit message: 秋の干渉スペシャル
Parts:
- moved LS1 43.8 mm to (513.7, 533.9)
- moved C18 30.0 mm to (520.9, 536.5)
- moved C17 29.8 mm to (520.9, 533.7)
- moved C19 17.4 mm to (520.9, 491.7)
- moved C20 16.0 mm to (521.0, 494.6)
- moved C25 15.2 mm to (525.2, 533.8), turned to 180 degrees
- moved R1 11.9 mm to (522.1, 508.1), turned to 180 degrees
- moved B1 11.7 mm to (522.0, 505.2)
- moved C26 10.6 mm to (525.8, 493.0), turned to 90 degrees
- moved C24 3.51 mm to (526.9, 505.3), turned to 90 degrees
- moved C23 2.67 mm to (529.7, 505.3), turned to -90 degrees
Connections:
- C25 pad 1: IMU_5V -> VCC
- C26 pad 1: IMU_5V -> VCC
- RP2040_Zero1 pad 1: unconnected-(RP2040_Zero1-0-Pad1) -> RP1_TX
- RP2040_Zero1 pad 13: RP1_TX -> OUT_TX
- RP2040_Zero1 pad 14: RP1_RX -> OUT_RX
- RP2040_Zero1 pad 2: unconnected-(RP2040_Zero1-1-Pad2) -> RP1_RX
- RP2040_Zero1 pad 3: unconnected-(RP2040_Zero1-2-Pad3) -> Conp_PWM
- RP2040_Zero2 pad 1: OUT_TX -> unconnected-(RP2040_Zero2-0-Pad1)
- RP2040_Zero2 pad 2: OUT_RX -> unconnected-(RP2040_Zero2-1-Pad2)
Routing:
- net GND: track 829.3 -> 927.3 mm, vias 64 -> 68
- net IMU_5V: track 0.00 -> 89.6 mm, vias 0 -> 6
- net VCC: track 729.1 -> 818.4 mm, vias 0 -> 23
- net RP1_RX: track 0.00 -> 83.4 mm, vias 0 -> 4
- net RP1_TX: track 0.00 -> 79.3 mm, vias 0 -> 4
- net conp_+: track 95.2 -> 139.8 mm, vias 32 -> 33
- net unconnected-(RP2040_Zero1-5-Pad6): track 0.00 -> 33.0 mm, vias 0 -> 2
- net 12: track 3.84 -> 34.9 mm, vias 0 -> 1
- net 32: track 3.84 -> 34.8 mm
- net unconnected-(RP2040_Zero1-6-Pad7): track 0.00 -> 29.6 mm, vias 0 -> 2
- net unconnected-(RP2040_Zero2-14-Pad15): track 0.00 -> 27.6 mm, vias 0 -> 1
- net 11: track 3.08 -> 29.9 mm, vias 0 -> 1
- net Net-(RP2040_Zero1-7): track 0.00 -> 26.4 mm, vias 0 -> 1
- net OUT_TX: track 0.00 -> 25.7 mm, vias 0 -> 1
- net 10: track 3.84 -> 29.0 mm, vias 0 -> 1
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
Commit message: 半球終了
Parts:
- moved B2 102.2 mm to (539.6, 535.5), turned to -90 degrees
- moved RV1 100.1 mm to (532.5, 541.1), turned to -90 degrees
- moved LS1 49.0 mm to (548.0, 498.8)
- moved C23 7.93 mm to (521.8, 504.5), turned to 180 degrees
- moved C24 6.35 mm to (521.8, 501.4), turned to 180 degrees
- moved J2 4.43 mm to (471.9, 548.1), turned to 63.52 degrees
- moved B1 3.82 mm to (524.0, 508.5), turned to -90 degrees
- moved C17 3.02 mm to (523.1, 535.8)
- moved C18 3.02 mm to (523.1, 538.6)
- moved C25 3.02 mm to (527.4, 535.9)
- moved C26 2.37 mm to (524.9, 490.9), turned to -90 degrees
- moved D33 1.33 mm to (518.2, 553.7)
- moved J3 1.26 mm to (515.1, 558.0)
- moved R1 1.10 mm to (521.0, 508.4), turned to 90 degrees
- moved RP2040_Zero1 1.00 mm to (530.0, 522.0)
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Connections:
- RP2040_Zero1 pad 10: unconnected-(RP2040_Zero1-9-Pad10) -> 24
- RP2040_Zero1 pad 11: unconnected-(RP2040_Zero1-10-Pad11) -> 26
- RP2040_Zero1 pad 12: unconnected-(RP2040_Zero1-11-Pad12) -> 29
- RP2040_Zero1 pad 13: OUT_TX -> 30
- RP2040_Zero1 pad 14: OUT_RX -> 27
- RP2040_Zero1 pad 15: unconnected-(RP2040_Zero1-14-Pad15) -> 23
- RP2040_Zero1 pad 16: unconnected-(RP2040_Zero1-15-Pad16) -> 22
- RP2040_Zero1 pad 17: unconnected-(RP2040_Zero1-26-Pad17) -> 21
- RP2040_Zero1 pad 19: unconnected-(RP2040_Zero1-28-Pad19) -> OUT_TX
- RP2040_Zero1 pad 20: unconnected-(RP2040_Zero1-29-Pad20) -> OUT_RX
- RP2040_Zero1 pad 4: unconnected-(RP2040_Zero1-3-Pad4) -> 25
- RP2040_Zero1 pad 5: unconnected-(RP2040_Zero1-4-Pad5) -> 28
- RP2040_Zero1 pad 6: unconnected-(RP2040_Zero1-5-Pad6) -> 31
- RP2040_Zero1 pad 7: unconnected-(RP2040_Zero1-6-Pad7) -> 32
- RP2040_Zero1 pad 8: Net-(RP2040_Zero1-7) -> 1
- RP2040_Zero1 pad 9: unconnected-(RP2040_Zero1-8-Pad9) -> 2
- RP2040_Zero2 pad 19: unconnected-(RP2040_Zero2-28-Pad19) -> RP1_RX
- RP2040_Zero2 pad 20: unconnected-(RP2040_Zero2-29-Pad20) -> RP1_TX
- RP2040_Zero2 pad 5: RP1_RX -> unconnected-(RP2040_Zero2-4-Pad5)
- RP2040_Zero2 pad 6: RP1_TX -> unconnected-(RP2040_Zero2-5-Pad6)
Routing:
- net VCC: track 818.4 -> 746.1 mm, vias 23 -> 17
- net 25: track 3.08 -> 66.7 mm, vias 0 -> 3
- net IMU_5V: track 89.6 -> 33.6 mm, vias 6 -> 3
- net RP1_RX: track 83.4 -> 29.2 mm, vias 4 -> 0
- net 24: track 3.75 -> 57.0 mm, vias 0 -> 5
- net 21: track 3.08 -> 53.2 mm, vias 0 -> 7
- net RP1_TX: track 79.3 -> 29.2 mm, vias 4 -> 0
- net GND: track 927.3 -> 877.3 mm, vias 68 -> 63
- net 22: track 3.84 -> 49.1 mm, vias 0 -> 4
- net 23: track 3.08 -> 44.8 mm, vias 0 -> 3
- net unconnected-(RP2040_Zero1-5-Pad6): track 33.0 -> 0.00 mm, vias 2 -> 0
- net 26: track 3.94 -> 36.3 mm, vias 0 -> 3
- net 28: track 6.90 -> 38.0 mm, vias 1 -> 3
- net 12: track 34.9 -> 3.95 mm, vias 1 -> 0
- net unconnected-(RP2040_Zero1-6-Pad7): track 29.6 -> 0.00 mm, vias 2 -> 0
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Other:
- outline, holes or cut-outs redrawn

Commit message: 平滑化用コンデンサTHTにした、0.1uFと10kΩ？
Parts:
- C24: footprint Capacitor_SMD:C_0603_1608Metric_Pad1.08x0.95mm_HandSolder -> Capacitor_THT:C_Rect_L7.0mm_W2.0mm_P5.00mm
- moved LS1 38.7 mm to (533.4, 534.7), turned to -90 degrees
- moved C24 1.77 mm to (520.2, 502.1), turned to 90 degrees
- moved C23 0.75 mm to (521.9, 505.3)
Connections:
- LS1 pad 1: unconnected-(LS1-Pad1) -> Net-(RP2040_Zero1-27)
- LS1 pad 2: unconnected-(LS1-Pad2) -> GND
- RP2040_Zero1 pad 18: unconnected-(RP2040_Zero1-27-Pad18) -> Net-(RP2040_Zero1-27)
- RP2040_Zero2 pad 15: unconnected-(RP2040_Zero2-14-Pad15) -> 3
- RP2040_Zero2 pad 16: unconnected-(RP2040_Zero2-15-Pad16) -> 4
- RP2040_Zero2 pad 17: unconnected-(RP2040_Zero2-26-Pad17) -> 5
- RP2040_Zero2 pad 18: unconnected-(RP2040_Zero2-27-Pad18) -> 6
Routing:
- net IMU_5V: track 33.6 -> 131.9 mm, vias 3 -> 4
- net GND: track 877.3 -> 968.4 mm, vias 63 -> 64
- net 6: track 4.61 -> 58.8 mm, vias 0 -> 1
- net unconnected-(RP2040_Zero2-9-Pad10): track 0.00 -> 33.8 mm, vias 0 -> 1
- net 5: track 10.8 -> 43.7 mm, vias 0 -> 1
- net unconnected-(RP2040_Zero2-10-Pad11): track 0.00 -> 29.3 mm, vias 0 -> 1
- net 4: track 6.64 -> 33.8 mm, vias 0 -> 1
- net unconnected-(RP2040_Zero2-12-Pad13): track 0.00 -> 22.6 mm, vias 0 -> 1
- net 3: track 3.08 -> 23.7 mm, vias 0 -> 1
- net unconnected-(RP2040_Zero2-13-Pad14): track 0.00 -> 18.2 mm, vias 0 -> 1
- net unconnected-(RP2040_Zero2-8-Pad9): track 0.03 -> 7.74 mm, vias 0 -> 1
- net Net-(RP2040_Zero1-27): track 0.00 -> 4.12 mm
- net unconnected-(RP2040_Zero2-11-Pad12): track 0.00 -> 2.92 mm, vias 0 -> 1
- net VCC: track 746.1 -> 743.6 mm
- net 2: track 46.2 -> 43.9 mm
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
Commit message: 配線終了
Connections:
- RP2040_Zero2 pad 1: unconnected-(RP2040_Zero2-0-Pad1) -> 10
- RP2040_Zero2 pad 10: unconnected-(RP2040_Zero2-9-Pad10) -> 7
- RP2040_Zero2 pad 11: unconnected-(RP2040_Zero2-10-Pad11) -> 8
- RP2040_Zero2 pad 12: unconnected-(RP2040_Zero2-11-Pad12) -> 11
- RP2040_Zero2 pad 13: unconnected-(RP2040_Zero2-12-Pad13) -> 13
- RP2040_Zero2 pad 14: unconnected-(RP2040_Zero2-13-Pad14) -> 12
- RP2040_Zero2 pad 2: unconnected-(RP2040_Zero2-1-Pad2) -> 9
- RP2040_Zero2 pad 3: unconnected-(RP2040_Zero2-2-Pad3) -> 19
- RP2040_Zero2 pad 4: unconnected-(RP2040_Zero2-3-Pad4) -> 17
- RP2040_Zero2 pad 5: unconnected-(RP2040_Zero2-4-Pad5) -> 15
- RP2040_Zero2 pad 6: unconnected-(RP2040_Zero2-5-Pad6) -> 20
- RP2040_Zero2 pad 7: unconnected-(RP2040_Zero2-6-Pad7) -> 18
- RP2040_Zero2 pad 8: Net-(RP2040_Zero2-7) -> 16
- RP2040_Zero2 pad 9: unconnected-(RP2040_Zero2-8-Pad9) -> 14
Routing:
- net 11: track 3.08 -> 73.5 mm, vias 0 -> 3
- net 12: track 3.84 -> 73.9 mm, vias 0 -> 6
- net 13: track 3.08 -> 66.8 mm, vias 0 -> 3
- net 8: track 5.44 -> 67.9 mm, vias 1 -> 2
- net 7: track 3.08 -> 54.8 mm, vias 0 -> 1
- net 14: track 3.84 -> 54.1 mm, vias 0 -> 3
- net 16: track 3.84 -> 43.0 mm, vias 0 -> 3
- net 9: track 3.08 -> 39.7 mm, vias 0 -> 1
- net 15: track 3.08 -> 38.8 mm, vias 0 -> 1
- net 19: track 3.08 -> 38.2 mm, vias 0 -> 1
- net 17: track 3.08 -> 36.9 mm, vias 0 -> 1
- net unconnected-(RP2040_Zero2-9-Pad10): track 33.8 -> 0.00 mm, vias 1 -> 0
- net 20: track 3.84 -> 37.5 mm, vias 0 -> 3
- net 18: track 3.84 -> 33.9 mm, vias 0 -> 3
- net unconnected-(RP2040_Zero2-10-Pad11): track 29.3 -> 0.00 mm, vias 1 -> 0
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Other:
- outline, holes or cut-outs redrawn

Commit message: 塗りつぶしまで
Routing:
- net VCC: track 728.4 -> 779.5 mm, vias 17 -> 19
- net GND: track 968.7 -> 999.1 mm, vias 58 -> 103
- net Net-(J1-Pin_1): track 36.7 -> 34.0 mm
- net IMU_5V: track 131.9 -> 129.8 mm
- net 3: track 23.7 -> 21.6 mm
- net 21: track 53.2 -> 51.3 mm
- net 12: track 73.9 -> 72.0 mm
- net 27: track 22.3 -> 20.5 mm
- net 24: track 57.0 -> 55.5 mm
- net 25: track 66.7 -> 65.3 mm
- net 22: track 49.1 -> 47.7 mm
- net 19: track 38.2 -> 37.5 mm
- net 8: track 67.9 -> 67.2 mm
- net OUT_TX: track 26.0 -> 25.3 mm
- net 7: track 54.8 -> 54.2 mm
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- added copper zone on B.Cu, net GND
- added copper zone on F.Cu, net GND
