File: KiCad/prot4/ネット減らしたい/prot4(カクカク配線修正前)/prot4.kicad_pcb (KiCad board)
At the start: 2 copper layers, 140 x 140 mm, 217 parts, among them J1 Conn_01x02_Socket, J2 LED_SW, J3 Conn_01x04_Socket, Q1 Q_Photo_NPN, Q10 Q_Photo_NPN, Q11 Q_Photo_NPN, Q12 Q_Photo_NPN, Q13 Q_Photo_NPN, Q14 Q_Photo_NPN, Q15 Q_Photo_NPN, Q16 Q_Photo_NPN, Q17 Q_Photo_NPN, Q18 Q_Photo_NPN, Q19 Q_Photo_NPN, Q2 Q_Photo_NPN, Q20 Q_Photo_NPN, Q21 Q_Photo_NPN, Q22 Q_Photo_NPN, Q23 Q_Photo_NPN, Q24 Q_Photo_NPN, Q25 Q_Photo_NPN, Q26 Q_Photo_NPN, Q27 Q_Photo_NPN, Q28 Q_Photo_NPN, Q29 Q_Photo_NPN, Q3 Q_Photo_NPN, Q30 Q_Photo_NPN, Q31 Q_Photo_NPN, Q32 Q_Photo_NPN, Q4 Q_Photo_NPN, Q5 Q_Photo_NPN, Q6 Q_Photo_NPN, Q7 Q_Photo_NPN, Q8 Q_Photo_NPN, Q9 Q_Photo_NPN, U1 LM393, U10 LM393, U11 LM393, U12 LM393, U13 LM393, U14 LM393, U15 LM393, U16 LM393, U2 LM393, U3 LM393, U4 LM393, U5 LM393, U6 LM393, U7 LM393, U8 LM393, U9 LM393

Commit message: 発注
Routing:
- net VCC: track 726.3 -> 779.5 mm, vias 22 -> 19
- net GND: track 1008.6 -> 999.1 mm, vias 160 -> 103
- net Net-(Q21-E): track 19.9 -> 21.8 mm
- net Net-(Q13-E): track 19.9 -> 21.8 mm
- net Net-(Q5-E): track 19.9 -> 21.8 mm
- net Net-(Q25-E): track 19.9 -> 21.8 mm
- net Net-(Q9-E): track 19.9 -> 21.8 mm
- net Net-(Q17-E): track 19.9 -> 21.8 mm
- net Net-(Q19-E): track 19.9 -> 21.8 mm
- net Net-(Q11-E): track 19.9 -> 21.8 mm
- net Net-(Q23-E): track 19.9 -> 21.8 mm
- net Net-(Q15-E): track 19.9 -> 21.8 mm
- net Net-(Q7-E): track 19.9 -> 21.8 mm
- net Net-(Q27-E): track 19.9 -> 21.8 mm
- net Net-(Q31-E): track 19.9 -> 21.8 mm
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